File: tempomat/circuits/tempomat/tempomat_main_board.sch (EAGLE design)
At the start: 66 parts, among them Q1 2N4033, Q2 BC489, Q4 2N4416, Q5 MPSA13, Q8 MPSA13, T1 TIP122, T2 TIP32C, T2-TIP127 BDX54, T3 TIP122, T4-TIP127 BDX54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

Commit message: reg save
Parts:
- removed R37: 27 k, resistor:R-EU_0204/2V
- added C3: 1n, resistor:C-EU025-060X050
- added C31, C8: 100n, resistor:C-EU025-060X050
- added D5, D6: 1N4004, diode:1N4004
- added R38, R40: 2.7k, resistor:R-EU_0204/2V
- added R4: 10k, resistor:R-EU_0204/2V
- added R44-?: 220, resistor:R-EU_0204/2V
- added R5: 180k, resistor:R-EU_0204/2V
- added U2-LM2903N: OPA2650E, burr-brown:OPA2650E
- renumbered Q2 to Q3
Connections:
- removed net N$29: D10.A, Q3.E
- new net N$47: Q4.B, R38.1
- new net N$48: C31.2, R32.2, R38.2
- new net N$49: Q8.B, R40.1
- new net N$50: C8.2, D5.C
- new net N$51: D5.A, R44-?.2
- new net N$52: C3.2, R44-?.1
- new net N$53: C15.-, C3.1
- new net N$54: C15.+, D6.A, U2-LM2903NB.+IN
- new net N$55: D6.C, R5.2
- net AGND: now also C31.1, C8.1, D10.A, Q3.E
- net N$30: no longer Q3.C
- net N$38: now also R40.2; no longer R32.2
- net N$45: no longer R37.1
- net N$46: no longer R37.2
Other:
- note added: "1"
- note added: "10"
- note added: "11"
- note added: "19"
- note added: "br/we"
- note added: "mps 5172"
- note removed: "mips 5172"
- moved on the sheet: C15, R32

Commit message: reg save
Parts:
- added C4, C9: 100n, resistor:C-EU025-060X050
- added D8: 1N4004, diode:1N4004
- added Q2: (no value), special:XTAL
- added R13: 100k, resistor:R-EU_0204/2V
- added R42, R43: 39k, resistor:R-EU_0204/2V
- added R6: 2k, resistor:R-EU_0204/2V
Connections:
- new net N$29: C4.2, Q2.1
- new net N$56: C9.2, Q2.2, R42.1, R43.1
- net AGND: now also C35.1, C4.1, C9.1, R14-R15_BETWEEN.2, R6.1
- net N$24: now also C35.2, D8.A, D8.C, R13.2; no longer C35.1
- net N$25: now also R13.1, R6.2; no longer C35.2, R14-R15_BETWEEN.2
Other:
- note added: "2"
- moved on the sheet: C35
Changed lines of the file:
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@@
 <part name="R4" library="resistor" deviceset="R-EU_" device="0204/2V" value="10k"/>
 <part name="SUPPLY19" library="supply2" deviceset="AGND" device=""/>
+<part name="Q2" library="special" deviceset="XTAL" device=""/>
+<part name="SUPPLY20" library="supply2" deviceset="AGND" device=""/>
+<part name="C4" library="resistor" deviceset="C-EU" device="025-060X050" value="100n"/>
+<part name="C9" library="resistor" deviceset="C-EU" device="025-060X050" value="100n"/>
+<part name="R42" library="resistor" deviceset="R-EU_" device="0204/2V" value="39k"/>
+<part name="R43" library="resistor" deviceset="R-EU_" device="0204/2V" value="39k"/>
+<part name="SUPPLY21" library="supply2" deviceset="AGND" device=""/>
+<part name="D8" library="diode" deviceset="1N4004" device=""/>
+<part name="R13" library="resistor" deviceset="R-EU_" device="0204/2V" value="100k"/>
+<part name="R6" library="resistor" deviceset="R-EU_" device="0204/2V" value="2k"/>
+<part name="SUPPLY22" library="supply2" deviceset="AGND" device=""/>
 </parts>
 <sheets>
@@
 <text x="2.54" y="81.28" size="1.778" layer="91">br</text>
 <text x="-48.26" y="-99.06" size="1.778" layer="91">br</text>
-<text x="91.44" y="45.72" size="1.778" layer="91">1</text>
 <text x="121.92" y="45.72" size="1.778" layer="91">11</text>
 <text x="134.62" y="45.72" size="1.778" layer="91">5</text>
-<text x="63.5" y="45.72" size="1.778" layer="91">10</text>
+<text x="60.96" y="43.18" size="1.778" layer="91">10</text>
 <text x="58.42" y="68.58" size="1.778" layer="91">11</text>
+<text x="68.58" y="45.72" size="1.778" layer="91">2</text>
+<text x="81.28" y="45.72" size="1.778" layer="91">1</text>
+<text x="88.9" y="45.72" size="1.778" layer="91">2</text>
 </plain>
 <instances>
@@
 <instance part="SUPPLY7" gate="G$1" x="10.16" y="-33.02"/>
 <instance part="R14-R15_BETWEEN" gate="G$1" x="35.56" y="-33.02" rot="R90"/>
-<instance part="C35" gate="G$1" x="58.42" y="40.64" rot="R90"/>
+<instance part="C35" gate="G$1" x="55.88" y="38.1" rot="R90"/>
 <instance part="SUPPLY8" gate="G$1" x="58.42" y="-43.18"/>
 <instance part="R30" gate="G$1" x="132.08" y="-7.62" rot="R90"/>
@@
 <instance part="R5" gate="G$1" x="96.52" y="-58.42" rot="R90"/>
 <instance part="R4" gate="G$1" x="96.52" y="-43.18" rot="R90"/>
-<instance part="SUPPLY19" gate="G$1" x="91.44" y="0"/>
+<instance part="SUPPLY19" gate="G$1" x="93.98" y="0"/>
+<instance part="Q2" gate="G$1" x="76.2" y="38.1"/>
+<instance part="SUPPLY20" gate="G$1" x="81.28" y="27.94"/>
+<instance part="C4" gate="G$1" x="68.58" y="33.02" rot="R180"/>
+<instance part="C9" gate="G$1" x="81.28" y="33.02" rot="R180"/>
+<instance part="R42" gate="G$1" x="81.28" y="43.18" rot="R90"/>
+<instance part="R43" gate="G$1" x="88.9" y="43.18" rot="R90"/>
+<instance part="SUPPLY21" gate="G$1" x="53.34" y="35.56"/>
+<instance part="D8" gate="1" x="78.74" y="12.7" rot="R180"/>
+<instance part="R13" gate="G$1" x="78.74" y="20.32" rot="R180"/>
+<instance part="R6" gate="G$1" x="93.98" y="15.24" rot="R180"/>
+<instance part="SUPPLY22" gate="G$1" x="99.06" y="12.7"/>
 </instances>
 <busses>
@@
 <pinref part="Q3" gate="G$1" pin="E"/>
 <wire x1="134.62" y1="-2.54" x2="144.78" y2="-2.54" width="0.1524" layer="91"/>
-<wire x1="106.68" y1="2.54" x2="91.44" y2="2.54" width="0.1524" layer="91"/>
-<wire x1="91.44" y1="2.54" x2="91.44" y2="48.26" width="0.1524" layer="91"/>
+<wire x1="106.68" y1="2.54" x2="93.98" y2="2.54" width="0.1524" layer="91"/>
 <pinref part="SUPPLY19" gate="G$1" pin="AGND"/>
-<junction x="91.44" y="2.54"/>
+<pinref part="R14-R15_BETWEEN" gate="G$1" pin="2"/>
+<wire x1="35.56" y1="-27.94" x2="35.56" y2="-10.16" width="0.1524" layer="91"/>
+<wire x1="35.56" y1="-10.16" x2="35.56" y2="25.4" width="0.1524" layer="91"/>
+<wire x1="35.56" y1="25.4" x2="55.88" y2="25.4" width="0.1524" layer="91"/>
+<wire x1="55.88" y1="25.4" x2="60.96" y2="25.4" width="0.1524" layer="91"/>
+<wire x1="35.56" y1="-10.16" x2="45.72" y2="-10.16" width="0.4064" layer="91"/>
+<wire x1="93.98" y1="2.54" x2="60.96" y2="2.54" width="0.1524" layer="91"/>
+<wire x1="60.96" y1="2.54" x2="60.96" y2="25.4" width="0.1524" layer="91"/>
+<wire x1="55.88" y1="25.4" x2="55.88" y2="38.1" width="0.1524" layer="91"/>
+</segment>
+<segment>
+<wire x1="68.58" y1="30.48" x2="81.28" y2="30.48" width="0.1524" layer="91"/>
+<pinref part="SUPPLY20" gate="G$1" pin="AGND"/>
+<pinref part="C4" gate="G$1" pin="1"/>
+<pinref part="C9" gate="G$1" pin="1"/>
+<junction x="81.28" y="30.48"/>
+<junction x="68.58" y="30.48"/>
+</segment>
+<segment>
+<pinref part="C35" gate="G$1" pin="1"/>
+<wire x1="53.34" y1="38.1" x2="53.34" y2="73.66" width="0.1524" layer="91"/>
+<wire x1="53.34" y1="73.66" x2="58.42" y2="73.66" width="0.1524" layer="91"/>
+<wire x1="58.42" y1="73.66" x2="58.42" y2="68.58" width="0.1524" layer="91"/>
+<pinref part="SUPPLY21" gate="G$1" pin="AGND"/>
+<junction x="53.34" y="38.1"/>
+</segment>
+<segment>
+<pinref part="R6" gate="G$1" pin="1"/>
+<pinref part="SUPPLY22" gate="G$1" pin="AGND"/>
 </segment>
 </net>
@@
 </segment>
 </net>
-<net name="N$25" class="0">
-<segment>
-<pinref part="C35" gate="G$1" pin="2"/>
-<wire x1="63.5" y1="40.64" x2="63.5" y2="48.26" width="0.1524" layer="91"/>
-<junction x="63.5" y="40.64"/>
-<pinref part="R14-R15_BETWEEN" gate="G$1" pin="2"/>
-<wire x1="35.56" y1="-27.94" x2="35.56" y2="-10.16" width="0.1524" layer="91"/>
-<wire x1="35.56" y1="-10.16" x2="35.56" y2="25.4" width="0.1524" layer="91"/>
-<wire x1="35.56" y1="25.4" x2="63.5" y2="25.4" width="0.1524" layer="91"/>
-<wire x1="63.5" y1="25.4" x2="63.5" y2="40.64" width="0.1524" layer="91"/>
-<wire x1="35.56" y1="-10.16" x2="45.72" y2="-10.16" width="0.4064" layer="91"/>
-</segment>
-</net>
-<net name="N$24" class="0">
-<segment>
-<pinref part="C35" gate="G$1" pin="1"/>
-<wire x1="55.88" y1="40.64" x2="53.34" y2="40.64" width="0.1524" layer="91"/>
-<wire x1="53.34" y1="40.64" x2="53.34" y2="73.66" width="0.1524" layer="91"/>
-<wire x1="53.34" y1="73.66" x2="58.42" y2="73.66" width="0.1524" layer="91"/>
-<wire x1="58.42" y1="73.66" x2="58.42" y2="68.58" width="0.1524" layer="91"/>
-</segment>
-</net>
 <net name="N$18" class="0">
 <segment>
@@
 </segment>
 </net>
+<net name="N$29" class="0">
+<segment>
+<pinref part="Q2" gate="G$1" pin="1"/>
+<wire x1="71.12" y1="38.1" x2="68.58" y2="38.1" width="0.1524" layer="91"/>
+<pinref part="C4" gate="G$1" pin="2"/>
+<wire x1="68.58" y1="38.1" x2="68.58" y2="48.26" width="0.1524" layer="91"/>
+<junction x="68.58" y="38.1"/>
+</segment>
+</net>
+<net name="N$56" class="0">
+<segment>
+<pinref part="Q2" gate="G$1" pin="2"/>
+<pinref part="C9" gate="G$1" pin="2"/>
+<wire x1="81.28" y1="38.1" x2="88.9" y2="38.1" width="0.1524" layer="91"/>
+<pinref part="R42" gate="G$1" pin="1"/>
+<junction x="81.28" y="38.1"/>
+<pinref part="R43" gate="G$1" pin="1"/>
+</segment>
+</net>
+<net name="N$24" class="0">
+<segment>
+<pinref part="C35" gate="G$1" pin="2"/>
+<wire x1="60.96" y1="38.1" x2="60.96" y2="48.26" width="0.1524" layer="91"/>
+<wire x1="60.96" y1="38.1" x2="60.96" y2="27.94" width="0.1524" layer="91"/>
+<wire x1="60.96" y1="27.94" x2="71.12" y2="27.94" width="0.1524" layer="91"/>
+<wire x1="71.12" y1="27.94" x2="71.12" y2="20.32" width="0.1524" layer="91"/>
+<pinref part="D8" gate="1" pin="A"/>
+<pinref part="D8" gate="1" pin="C"/>
+<wire x1="71.12" y1="20.32" x2="71.12" y2="12.7" width="0.1524" layer="91"/>
+<wire x1="76.2" y1="12.7" x2="81.28" y2="12.7" width="0.1524" layer="91"/>
+<wire x1="76.2" y1="12.7" x2="71.12" y2="12.7" width="0.1524" layer="91"/>
+<pinref part="R13" gate="G$1" pin="2"/>
+<wire x1="71.12" y1="20.32" x2="73.66" y2="20.32" width="0.1524" layer="91"/>
+</segment>
+</net>
+<net name="N$25" class="0">
+<segment>
+<pinref part="R13" gate="G$1" pin="1"/>
+<wire x1="83.82" y1="20.32" x2="88.9" y2="20.32" width="0.1524" layer="91"/>
+<wire x1="88.9" y1="20.32" x2="88.9" y2="15.24" width="0.1524" layer="91"/>
+<pinref part="R6" gate="G$1" pin="2"/>
+</segment>
+</net>

Commit message: reg save
Connections:
- removed net N$48: C31.2, R32.2, R38.2
- new net N$57: R38.2
- net AGND: no longer C11.+, C37.1
- net N$28: now also R32.1; no longer C37.2
- net N$30: now also R4.2; no longer R32.1, U4_XOR-D.I1
- net N$55: now also R4.1
Other:
- note added: "14"
- moved on the sheet: C11, C31, C37, R32, U-XY-A, U-XY-B
