File: tempomat/circuits/tempomat/tempix_main.sch (EAGLE design)
At the start: 4 parts

Commit message: reg save
Parts:
- added SV4: (no value), con-amp-mt:L07P
Other:
- note added: "Clu1"
- note added: "Clu2"
- note added: "Mot1"
- note added: "Mot2"
- note added: "NC"
- note added: "Pot+"
- note added: "Pot-"
- note added: "PotS"
- moved on the sheet: C1, SV1-1, SV1-2, SV1-3, SV1-4, SV1-5, SV2-1, SV2-2, SV2-3, SV2-4, SV2-5, SV3-1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
