File: nixi/nixi/nixi-test-board.sch (EAGLE design)
At the start: 0 parts

Commit message: reg save
Parts:
- added C1, C2, C3: (no value), resistor:CPOL-EU139CLL-2W
- added D1: 1N4942, diode:1N4942
- added IC1: 7805T, linear:7805T
- added IC2: TINY15LP, atmel:TINY15LP
- added L1: (no value), inductor-neosid:U15-CHOKE
- added POWER: (no value), con-amp-mt:L02P
- added Q1: MRF136, transistor-fet:MRF136
- added R1, R2, R3: (no value), resistor:R-EU_0207/5V
- added SX1: VT9-PT, belton-engineering:VT9-PT
Connections:
- new net +12V: C3.+, IC1.VI, POWER-1.S
- new net +5V: C2.+, IC1.VO
- new net GND: IC1.GND, POWER-2.S, SX1.1
Changed lines of the file:
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@@
 <grid distance="0.1" unitdist="inch" unit="inch" style="lines" multiple="1" display="no" altdistance="0.01" altunitdist="inch" altunit="inch"/>
 <layers>
+<layer number="1" name="Top" color="4" fill="1" visible="no" active="no"/>
+<layer number="2" name="Route2" color="1" fill="3" visible="no" active="no"/>
+<layer number="3" name="Route3" color="4" fill="3" visible="no" active="no"/>
+<layer number="4" name="Route4" color="1" fill="4" visible="no" active="no"/>
+<layer number="5" name="Route5" color="4" fill="4" visible="no" active="no"/>
+<layer number="6" name="Route6" color="1" fill="8" visible="no" active="no"/>
+<layer number="7" name="Route7" color="4" fill="8" visible="no" active="no"/>
+<layer number="8" name="Route8" color="1" fill="2" visible="no" active="no"/>
+<layer number="9" name="Route9" color="4" fill="2" visible="no" active="no"/>
+<layer number="10" name="Route10" color="1" fill="7" visible="no" active="no"/>
+<layer number="11" name="Route11" color="4" fill="7" visible="no" active="no"/>
+<layer number="12" name="Route12" color="1" fill="5" visible="no" active="no"/>
+<layer number="13" name="Route13" color="4" fill="5" visible="no" active="no"/>
+<layer number="14" name="Route14" color="1" fill="6" visible="no" active="no"/>
+<layer number="15" name="Route15" color="4" fill="6" visible="no" active="no"/>
+<layer number="16" name="Bottom" color="1" fill="1" visible="no" active="no"/>
+<layer number="17" name="Pads" color="2" fill="1" visible="no" active="no"/>
+<layer number="18" name="Vias" color="2" fill="1" visible="no" active="no"/>
+<layer number="19" name="Unrouted" color="6" fill="1" visible="no" active="no"/>
+<layer number="20" name="Dimension" color="15" fill="1" visible="no" active="no"/>
+<layer number="21" name="tPlace" color="7" fill="1" visible="no" active="no"/>
+<layer number="22" name="bPlace" color="7" fill="1" visible="no" active="no"/>
+<layer number="23" name="tOrigins" color="15" fill="1" visible="no" active="no"/>
+<layer number="24" name="bOrigins" color="15" fill="1" visible="no" active="no"/>
+<layer number="25" name="tNames" color="7" fill="1" visible="no" active="no"/>
+<layer number="26" name="bNames" color="7" fill="1" visible="no" active="no"/>
+<layer number="27" name="tValues" color="7" fill="1" visible="no" active="no"/>
+<layer number="28" name="bValues" color="7" fill="1" visible="no" active="no"/>
+<layer number="29" name="tStop" color="7" fill="3" visible="no" active="no"/>
+<layer number="30" name="bStop" color="7" fill="6" visible="no" active="no"/>
+<layer number="31" name="tCream" color="7" fill="4" visible="no" active="no"/>
+<layer number="32" name="bCream" color="7" fill="5" visible="no" active="no"/>
+<layer number="33" name="tFinish" color="6" fill="3" visible="no" active="no"/>
+<layer number="34" name="bFinish" color="6" fill="6" visible="no" active="no"/>
+<layer number="35" name="tGlue" color="7" fill="4" visible="no" active="no"/>
+<layer number="36" name="bGlue" color="7" fill="5" visible="no" active="no"/>
+<layer number="37" name="tTest" color="7" fill="1" visible="no" active="no"/>
+<layer number="38" name="bTest" color="7" fill="1" visible="no" active="no"/>
+<layer number="39" name="tKeepout" color="4" fill="11" visible="no" active="no"/>
+<layer number="40" name="bKeepout" color="1" fill="11" visible="no" active="no"/>
+<layer number="41" name="tRestrict" color="4" fill="10" visible="no" active="no"/>
+<layer number="42" name="bRestrict" color="1" fill="10" visible="no" active="no"/>
+<layer number="43" name="vRestrict" color="2" fill="10" visible="no" active="no"/>
+<layer number="44" name="Drills" color="7" fill="1" visible="no" active="no"/>
+<layer number="45" name="Holes" color="7" fill="1" visible="no" active="no"/>
+<layer number="46" name="Milling" color="3" fill="1" visible="no" active="no"/>
+<layer number="47" name="Measures" color="7" fill="1" visible="no" active="no"/>
+<layer number="48" name="Document" color="7" fill="1" visible="no" active="no"/>
+<layer number="49" name="Reference" color="7" fill="1" visible="no" active="no"/>
+<layer number="51" name="tDocu" color="6" fill="9" visible="no" active="no"/>
+<layer number="52" name="bDocu" color="7" fill="1" visible="no" active="no"/>
 <layer number="90" name="Modules" color="5" fill="1" visible="yes" active="yes"/>
 <layer number="91" name="Nets" color="2" fill="1" visible="yes" active="yes"/>
@@
 <layer number="97" name="Info" color="7" fill="1" visible="yes" active="yes"/>
 <layer number="98" name="Guide" color="6" fill="1" visible="yes" active="yes"/>
+<layer number="99" name="SpiceOrder" color="5" fill="1" visible="yes" active="yes"/>
 </layers>
 <schematic xreflabel="%F%N/%S.%C%R" xrefpart="/%S.%C%R">
@@
 </classes>
 <parts>
+<part name="IC2" library="atmel" deviceset="TINY15L" device="P"/>
+<part name="SX1" library="belton-engineering" deviceset="VT9" device="-PT"/>
+<part name="IC1" library="linear" deviceset="78*" device="T" technology="05"/>
+<part name="POWER" library="con-amp-mt" deviceset="L02P" device=""/>
+<part name="SUPPLY1" library="supply2" deviceset="GND" device=""/>
+<part name="SUPPLY2" library="supply2" deviceset="+12V" device=""/>
+<part name="SUPPLY3" library="supply2" deviceset="+5V" device=""/>
+<part name="SUPPLY4" library="supply2" deviceset="+5V" device=""/>
+<part name="L1" library="inductor-neosid" deviceset="U15-" device="CHOKE"/>
+<part name="D1" library="diode" deviceset="1N4942" device=""/>
+<part name="C1" library="resistor" deviceset="CPOL-EU" device="139CLL-2W"/>
+<part name="C2" library="resistor" deviceset="CPOL-EU" device="139CLL-2W"/>
+<part name="C3" library="resistor" deviceset="CPOL-EU" device="139CLL-2W"/>
+<part name="R1" library="resistor" deviceset="R-EU_" device="0207/5V"/>
+<part name="R2" library="resistor" deviceset="R-EU_" device="0207/5V"/>
+<part name="R3" library="resistor" deviceset="R-EU_" device="0207/5V"/>
+<part name="Q1" library="transistor-fet" deviceset="MRF136" device=""/>
 </parts>
 <sheets>
@@
 </plain>
 <instances>
+<instance part="IC2" gate="G$1" x="22.86" y="48.26"/>
+<instance part="SX1" gate="G$1" x="116.84" y="68.58"/>
+<instance part="IC1" gate="A1" x="17.78" y="81.28"/>
+<instance part="POWER" gate="-1" x="-33.02" y="88.9"/>
+<instance part="POWER" gate="-2" x="-33.02" y="83.82"/>
+<instance part="SUPPLY1" gate="GND" x="-7.62" y="38.1"/>
+<instance part="SUPPLY2" gate="+12V" x="-22.86" y="91.44"/>
+<instance part="SUPPLY3" gate="+5V" x="38.1" y="83.82"/>
+<instance part="SUPPLY4" gate="+5V" x="2.54" y="45.72"/>
+<instance part="L1" gate="G$1" x="81.28" y="20.32"/>
+<instance part="D1" gate="1" x="106.68" y="20.32"/>
+<instance part="C1" gate="G$1" x="132.08" y="17.78"/>
+<instance part="C2" gate="G$1" x="33.02" y="78.74"/>
+<instance part="C3" gate="G$1" x="2.54" y="78.74"/>
+<instance part="R1" gate="G$1" x="91.44" y="50.8"/>
+<instance part="R2" gate="G$1" x="73.66" y="60.96"/>
+<instance part="R3" gate="G$1" x="60.96" y="60.96"/>
+<instance part="Q1" gate="G$1" x="162.56" y="53.34"/>
 </instances>
 <busses>
 </busses>
 <nets>
+<net name="GND" class="0">
+<segment>
+<pinref part="POWER" gate="-2" pin="S"/>
+<wire x1="-27.94" y1="83.82" x2="-12.7" y2="83.82" width="0.1524" layer="91"/>
+<wire x1="-12.7" y1="83.82" x2="-12.7" y2="71.12" width="0.1524" layer="91"/>
+<wire x1="-12.7" y1="71.12" x2="17.78" y2="71.12" width="0.1524" layer="91"/>
+<pinref part="IC1" gate="A1" pin="GND"/>
+<wire x1="17.78" y1="71.12" x2="17.78" y2="73.66" width="0.1524" layer="91"/>
+<wire x1="17.78" y1="71.12" x2="96.52" y2="71.12" width="0.1524" layer="91"/>
+<wire x1="96.52" y1="71.12" x2="96.52" y2="78.74" width="0.1524" layer="91"/>
+<pinref part="SX1" gate="G$1" pin="1"/>
+<wire x1="96.52" y1="78.74" x2="109.22" y2="78.74" width="0.1524" layer="91"/>
+<wire x1="-12.7" y1="71.12" x2="-12.7" y2="40.64" width="0.1524" layer="91"/>
+<wire x1="-12.7" y1="40.64" x2="-7.62" y2="40.64" width="0.1524" layer="91"/>
+<pinref part="SUPPLY1" gate="GND" pin="GND"/>
+<wire x1="-7.62" y1="40.64" x2="7.62" y2="40.64" width="0.1524" layer="91"/>
+<junction x="-7.62" y="40.64"/>
+</segment>
+</net>
+<net name="+12V" class="0">
+<segment>
+<pinref part="POWER" gate="-1" pin="S"/>
+<wire x1="-27.94" y1="88.9" x2="-22.86" y2="88.9" width="0.1524" layer="91"/>
+<wire x1="-22.86" y1="88.9" x2="-10.16" y2="88.9" width="0.1524" layer="91"/>
+<wire x1="-10.16" y1="88.9" x2="-10.16" y2="81.28" width="0.1524" layer="91"/>
+<pinref part="IC1" gate="A1" pin="VI"/>
+<wire x1="-10.16" y1="81.28" x2="2.54" y2="81.28" width="0.1524" layer="91"/>
+<pinref part="SUPPLY2" gate="+12V" pin="+12V"/>
+<junction x="-22.86" y="88.9"/>
+<pinref part="C3" gate="G$1" pin="+"/>
+<wire x1="2.54" y1="81.28" x2="7.62" y2="81.28" width="0.1524" layer="91"/>
+<junction x="2.54" y="81.28"/>
+</segment>
+</net>
+<net name="+5V" class="0">
+<segment>
+<pinref part="IC1" gate="A1" pin="VO"/>
+<pinref part="SUPPLY3" gate="+5V" pin="+5V"/>
+<wire x1="27.94" y1="81.28" x2="33.02" y2="81.28" width="0.1524" layer="91"/>
+<pinref part="C2" gate="G$1" pin="+"/>
+<wire x1="33.02" y1="81.28" x2="38.1" y2="81.28" width="0.1524" layer="91"/>
+<junction x="33.02" y="81.28"/>
+</segment>
+<segment>
+<pinref part="SUPPLY4" gate="+5V" pin="+5V"/>
+<wire x1="2.54" y1="43.18" x2="7.62" y2="43.18" width="0.1524" layer="91"/>
+</segment>
+</net>
 </nets>
 </sheet>
