File: nixi/nixi/nixi-test-board.sch (EAGLE design)
At the start: 13 parts, among them IC1 7805T, IC2 TINY15LP, Q1 MRF136

Commit message: reg save
Parts:
- removed R1: (no value), resistor:R-EU_0207/5V
- added DEBUG, GND: (no value), con-amp-mt:L02P
- added R4: (no value), resistor:R-EU_0207/5V
- renumbered POWER to 12V
Connections:
- new net N$1: DEBUG-2.S, IC2.(ADC0)PB5
- new net N$2: L1.4, Q1.D
- new net N$3: C1.+, R3.1, SX1.2
- new net N$5: IC2.(ADC1)PB2, R2.1, R3.2
- new net N$6: IC2.(OCP)PB1, R4.1
- net +12V: now also D1.A, L1.1
- net GND: now also C1.-, C2.-, C3.-, DEBUG-1.S, GND-1.S, Q1.S, R2.2, R4.2; no longer 12V-2.S
Other:
- note added: "sense"
- moved on the sheet: C1, C2, C3, D1, L1, Q1, R2, R3

Commit message: reg save
Parts:
- removed R2: (no value), resistor:R-EU_0207/5V
- added RV1: (no value), resistor:R-TRIMM4G/J
- renumbered IC2 to IC2-ATTINY85, SX1 to NIXI-SOCKET
Connections:
- new net N$4: R3.2, RV1.A
- net GND: now also RV1.E; no longer R2.2
- net N$3: now also D1.C
- net N$5: now also RV1.S; no longer R2.1, R3.2
Other:
- note added: "HV 100-400 V"
- moved on the sheet: R4
Changed lines of the file:
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@@
 </classes>
 <parts>
-<part name="IC2" library="atmel" deviceset="TINY15L" device="P"/>
-<part name="SX1" library="belton-engineering" deviceset="VT9" device="-PT"/>
+<part name="IC2-ATTINY85" library="atmel" deviceset="TINY15L" device="P"/>
+<part name="NIXI-SOCKET" library="belton-engineering" deviceset="VT9" device="-PT"/>
 <part name="IC1" library="linear" deviceset="78*" device="T" technology="05"/>
 <part name="12V" library="con-amp-mt" deviceset="L02P" device=""/>
@@
 <part name="C2" library="resistor" deviceset="CPOL-EU" device="139CLL-2W"/>
 <part name="C3" library="resistor" deviceset="CPOL-EU" device="139CLL-2W"/>
-<part name="R2" library="resistor" deviceset="R-EU_" device="0207/5V"/>
 <part name="R3" library="resistor" deviceset="R-EU_" device="0207/5V"/>
 <part name="Q1" library="transistor-fet" deviceset="MRF136" device=""/>
@@
 <part name="R4" library="resistor" deviceset="R-EU_" device="0207/5V"/>
 <part name="GND" library="con-amp-mt" deviceset="L02P" device=""/>
+<part name="RV1" library="resistor" deviceset="R-TRIMM" device="4G/J"/>
 </parts>
 <sheets>
@@
 <plain>
 <text x="142.24" y="33.02" size="2.1844" layer="91">sense</text>
+<text x="134.62" y="45.72" size="1.9304" layer="91">HV 100-400 V</text>
 </plain>
 <instances>
-<instance part="IC2" gate="G$1" x="22.86" y="48.26"/>
-<instance part="SX1" gate="G$1" x="116.84" y="68.58"/>
+<instance part="IC2-ATTINY85" gate="G$1" x="22.86" y="48.26"/>
+<instance part="NIXI-SOCKET" gate="G$1" x="116.84" y="68.58"/>
 <instance part="IC1" gate="A1" x="17.78" y="81.28"/>
 <instance part="12V" gate="-1" x="-33.02" y="88.9"/>
@@
 <instance part="C2" gate="G$1" x="33.02" y="76.2"/>
 <instance part="C3" gate="G$1" x="2.54" y="76.2"/>
-<instance part="R2" gate="G$1" x="134.62" y="22.86" rot="R270"/>
 <instance part="R3" gate="G$1" x="134.62" y="35.56" rot="R270"/>
 <instance part="Q1" gate="G$1" x="76.2" y="30.48"/>
@@
 <instance part="SUPPLY5" gate="+12V" x="78.74" y="53.34"/>
 <instance part="SUPPLY7" gate="GND" x="134.62" y="12.7"/>
-<instance part="R4" gate="G$1" x="63.5" y="20.32" rot="R270"/>
+<instance part="R4" gate="G$1" x="63.5" y="22.86" rot="R270"/>
 <instance part="GND" gate="-1" x="-33.02" y="83.82"/>
+<instance part="RV1" gate="G$1" x="134.62" y="25.4"/>
 </instances>
 <busses>
@@
 <wire x1="33.02" y1="71.12" x2="96.52" y2="71.12" width="0.1524" layer="91"/>
 <wire x1="96.52" y1="71.12" x2="96.52" y2="78.74" width="0.1524" layer="91"/>
-<pinref part="SX1" gate="G$1" pin="1"/>
+<pinref part="NIXI-SOCKET" gate="G$1" pin="1"/>
 <wire x1="96.52" y1="78.74" x2="109.22" y2="78.74" width="0.1524" layer="91"/>
 <wire x1="-12.7" y1="71.12" x2="-12.7" y2="40.64" width="0.1524" layer="91"/>
@@
 </segment>
 <segment>
-<pinref part="R2" gate="G$1" pin="2"/>
-<pinref part="SUPPLY7" gate="GND" pin="GND"/>
 <pinref part="Q1" gate="G$1" pin="S"/>
 <wire x1="78.74" y1="22.86" x2="78.74" y2="17.78" width="0.1524" layer="91"/>
 <wire x1="78.74" y1="17.78" x2="114.3" y2="17.78" width="0.1524" layer="91"/>
-<wire x1="114.3" y1="17.78" x2="134.62" y2="17.78" width="0.1524" layer="91"/>
-<wire x1="134.62" y1="17.78" x2="134.62" y2="15.24" width="0.1524" layer="91"/>
-<wire x1="78.74" y1="17.78" x2="71.12" y2="17.78" width="0.1524" layer="91"/>
-<wire x1="71.12" y1="17.78" x2="71.12" y2="15.24" width="0.1524" layer="91"/>
-<pinref part="R4" gate="G$1" pin="2"/>
-<wire x1="71.12" y1="15.24" x2="63.5" y2="15.24" width="0.1524" layer="91"/>
 <pinref part="C1" gate="G$1" pin="-"/>
 <wire x1="114.3" y1="27.94" x2="114.3" y2="17.78" width="0.1524" layer="91"/>
+<pinref part="R4" gate="G$1" pin="2"/>
+<wire x1="63.5" y1="17.78" x2="78.74" y2="17.78" width="0.1524" layer="91"/>
+<wire x1="114.3" y1="17.78" x2="134.62" y2="17.78" width="0.1524" layer="91"/>
+<pinref part="SUPPLY7" gate="GND" pin="GND"/>
+<wire x1="134.62" y1="15.24" x2="134.62" y2="17.78" width="0.1524" layer="91"/>
+<pinref part="RV1" gate="G$1" pin="E"/>
+<wire x1="134.62" y1="20.32" x2="134.62" y2="17.78" width="0.1524" layer="91"/>
 </segment>
 </net>
@@
 <segment>
 <pinref part="DEBUG" gate="-2" pin="S"/>
-<pinref part="IC2" gate="G$1" pin="(ADC0)PB5"/>
+<pinref part="IC2-ATTINY85" gate="G$1" pin="(ADC0)PB5"/>
 <wire x1="45.72" y1="53.34" x2="40.64" y2="53.34" width="0.1524" layer="91"/>
 </segment>
@@
 <net name="N$3" class="0">
 <segment>
-<wire x1="106.68" y1="43.18" x2="114.3" y2="43.18" width="0.1524" layer="91"/>
+<wire x1="104.14" y1="43.18" x2="114.3" y2="43.18" width="0.1524" layer="91"/>
 <pinref part="R3" gate="G$1" pin="1"/>
 <wire x1="114.3" y1="43.18" x2="134.62" y2="43.18" width="0.1524" layer="91"/>
@@
 <wire x1="101.6" y1="68.58" x2="101.6" y2="66.04" width="0.1524" layer="91"/>
 <wire x1="101.6" y1="66.04" x2="101.6" y2="63.5" width="0.1524" layer="91"/>
-<pinref part="SX1" gate="G$1" pin="2"/>
+<pinref part="NIXI-SOCKET" gate="G$1" pin="2"/>
 <wire x1="101.6" y1="63.5" x2="101.6" y2="60.96" width="0.1524" layer="91"/>
 <wire x1="101.6" y1="60.96" x2="101.6" y2="58.42" width="0.1524" layer="91"/>
@@
 <wire x1="101.6" y1="60.96" x2="109.22" y2="60.96" width="0.1524" layer="91" style="shortdash"/>
 <wire x1="101.6" y1="58.42" x2="109.22" y2="58.42" width="0.1524" layer="91" style="shortdash"/>
+<pinref part="D1" gate="1" pin="C"/>
 </segment>
 </net>
@@
 <segment>
 <pinref part="R4" gate="G$1" pin="1"/>
-<wire x1="63.5" y1="25.4" x2="63.5" y2="27.94" width="0.1524" layer="91"/>
 <wire x1="63.5" y1="27.94" x2="73.66" y2="27.94" width="0.1524" layer="91"/>
-<pinref part="IC2" gate="G$1" pin="(OCP)PB1"/>
+<pinref part="IC2-ATTINY85" gate="G$1" pin="(OCP)PB1"/>
 <wire x1="40.64" y1="43.18" x2="63.5" y2="43.18" width="0.1524" layer="91"/>
 <wire x1="63.5" y1="43.18" x2="63.5" y2="27.94" width="0.1524" layer="91"/>
@@
 <net name="N$5" class="0">
 <segment>
-<pinref part="IC2" gate="G$1" pin="(ADC1)PB2"/>
+<pinref part="IC2-ATTINY85" gate="G$1" pin="(ADC1)PB2"/>
 <wire x1="40.64" y1="45.72" x2="48.26" y2="45.72" width="0.1524" layer="91"/>
 <wire x1="48.26" y1="45.72" x2="48.26" y2="40.64" width="0.1524" layer="91" curve="-180"/>
 <wire x1="48.26" y1="40.64" x2="48.26" y2="7.62" width="0.1524" layer="91"/>
 <wire x1="48.26" y1="7.62" x2="144.78" y2="7.62" width="0.1524" layer="91"/>
-<wire x1="144.78" y1="7.62" x2="144.78" y2="30.48" width="0.1524" layer="91"/>
+<pinref part="RV1" gate="G$1" pin="S"/>
+<wire x1="139.7" y1="25.4" x2="144.78" y2="25.4" width="0.1524" layer="91"/>
+<wire x1="144.78" y1="25.4" x2="144.78" y2="7.62" width="0.1524" layer="91"/>
+</segment>
+</net>
+<net name="N$4" class="0">
+<segment>
 <pinref part="R3" gate="G$1" pin="2"/>
-<pinref part="R2" gate="G$1" pin="1"/>
-<wire x1="134.62" y1="30.48" x2="134.62" y2="27.94" width="0.1524" layer="91"/>
-<wire x1="144.78" y1="30.48" x2="134.62" y2="30.48" width="0.1524" layer="91"/>
-</segment>
-</net>
+<pinref part="RV1" gate="G$1" pin="A"/>
+</segment>
+</net>
