File: nixi/nixi/nixi-test-board.sch (EAGLE design)
At the start: 15 parts, among them IC1 7805T, IC2-ATTINY85 TINY15LP, Q1 MRF136

Commit message: reg save
Other:
- note added: "Nixi Test"
Changed lines of the file:
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@@
 <text x="144.78" y="27.94" size="2.1844" layer="91">sense</text>
 <text x="134.62" y="45.72" size="1.9304" layer="91">HV 100-400 V</text>
+<text x="48.26" y="96.52" size="5.08" layer="91">Nixi  Test</text>
 </plain>
 <instances>

Commit message: reg save
Parts:
- removed R4: (no value), resistor:R-EU_0207/5V
- added Q2: 2N6107, transistor-pnp:2N6107
- added Q3: BC238, transistor-npn:BC238
- added R1, R2: (no value), resistor:R-EU_0207/5V
Connections:
- new net N$10: Q1.G, Q2.E, R1.2
- new net N$7: IC2-ATTINY85.(OCP)PB1, R2.1
- new net N$8: Q3.B, R2.2
- net GND: now also Q2.C, Q3.E, R1.1; no longer R4.2
- net N$3: now also NIXI-SOCKET.3, NIXI-SOCKET.4, NIXI-SOCKET.5, NIXI-SOCKET.6, NIXI-SOCKET.7, NIXI-SOCKET.8, NIXI-SOCKET.9
- net N$6: now also Q2.B, Q3.C; no longer IC2-ATTINY85.(OCP)PB1, R4.1
Other:
- moved on the sheet: C1, D1, L1, NIXI-SOCKET, Q1, R3, RV1

Commit message: reg save
Parts:
- R1: value (none) -> 3.3k
- R2: value (none) -> 1k
Connections:
- net +12V: now also R1.1
- net GND: no longer R1.1
Other:
- moved on the sheet: R1
Changed lines of the file:
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@@
 <part name="RV1" library="resistor" deviceset="R-TRIMM" device="4G/J"/>
 <part name="Q2" library="transistor-pnp" deviceset="2N6107" device=""/>
-<part name="R1" library="resistor" deviceset="R-EU_" device="0207/5V"/>
-<part name="R2" library="resistor" deviceset="R-EU_" device="0207/5V"/>
+<part name="R1" library="resistor" deviceset="R-EU_" device="0207/5V" value="3.3k"/>
+<part name="R2" library="resistor" deviceset="R-EU_" device="0207/5V" value="1k"/>
 <part name="Q3" library="transistor-npn" deviceset="BC238" device=""/>
 </parts>
@@
 <instance part="RV1" gate="G$1" x="170.18" y="25.4"/>
 <instance part="Q2" gate="G$1" x="96.52" y="22.86"/>
-<instance part="R1" gate="G$1" x="99.06" y="58.42" rot="R270"/>
+<instance part="R1" gate="G$1" x="99.06" y="40.64" rot="R270"/>
 <instance part="R2" gate="G$1" x="71.12" y="30.48" rot="R270"/>
 <instance part="Q3" gate="G$1" x="91.44" y="15.24"/>
@@
 <wire x1="17.78" y1="71.12" x2="17.78" y2="73.66" width="0.1524" layer="91"/>
 <wire x1="17.78" y1="71.12" x2="33.02" y2="71.12" width="0.1524" layer="91"/>
-<wire x1="33.02" y1="71.12" x2="99.06" y2="71.12" width="0.1524" layer="91"/>
-<wire x1="99.06" y1="71.12" x2="132.08" y2="71.12" width="0.1524" layer="91"/>
+<wire x1="33.02" y1="71.12" x2="132.08" y2="71.12" width="0.1524" layer="91"/>
 <wire x1="132.08" y1="71.12" x2="132.08" y2="78.74" width="0.1524" layer="91"/>
 <pinref part="NIXI-SOCKET" gate="G$1" pin="1"/>
@@
 <pinref part="C3" gate="G$1" pin="-"/>
 <pinref part="GND" gate="-1" pin="S"/>
-<pinref part="R1" gate="G$1" pin="1"/>
-<wire x1="99.06" y1="71.12" x2="99.06" y2="63.5" width="0.1524" layer="91"/>
 </segment>
 <segment>
@@
 <pinref part="D1" gate="1" pin="A"/>
 <wire x1="132.08" y1="43.18" x2="134.62" y2="43.18" width="0.1524" layer="91"/>
+<wire x1="114.3" y1="50.8" x2="99.06" y2="50.8" width="0.1524" layer="91"/>
+<pinref part="R1" gate="G$1" pin="1"/>
+<wire x1="99.06" y1="50.8" x2="99.06" y2="45.72" width="0.1524" layer="91"/>
 </segment>
 </net>
@@
 <wire x1="99.06" y1="27.94" x2="106.68" y2="27.94" width="0.1524" layer="91"/>
 <pinref part="R1" gate="G$1" pin="2"/>
-<wire x1="99.06" y1="53.34" x2="99.06" y2="27.94" width="0.1524" layer="91"/>
+<wire x1="99.06" y1="35.56" x2="99.06" y2="27.94" width="0.1524" layer="91"/>
 <pinref part="Q2" gate="G$1" pin="E"/>
 <junction x="99.06" y="27.94"/>

Commit message: reg save
Parts:
- renumbered IC2-ATTINY85 to STM32F103C8
Changed lines of the file:
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@@
 <layer number="48" name="Document" color="7" fill="1" visible="no" active="no"/>
 <layer number="49" name="Reference" color="7" fill="1" visible="no" active="no"/>
+<layer number="50" name="dxf" color="7" fill="1" visible="no" active="no"/>
 <layer number="51" name="tDocu" color="6" fill="9" visible="no" active="no"/>
 <layer number="52" name="bDocu" color="7" fill="1" visible="no" active="no"/>
@@
 <layer number="98" name="Guide" color="6" fill="1" visible="yes" active="yes"/>
 <layer number="99" name="SpiceOrder" color="5" fill="1" visible="yes" active="yes"/>
+<layer number="100" name="Muster" color="7" fill="1" visible="no" active="no"/>
+<layer number="101" name="Patch_Top" color="12" fill="4" visible="yes" active="yes"/>
+<layer number="116" name="Patch_BOT" color="9" fill="4" visible="yes" active="yes"/>
+<layer number="200" name="200bmp" color="1" fill="10" visible="no" active="no"/>
+<layer number="250" name="Descript" color="3" fill="1" visible="no" active="no"/>
+<layer number="251" name="SMDround" color="12" fill="11" visible="no" active="no"/>
+<layer number="254" name="cooling" color="7" fill="1" visible="yes" active="yes"/>
 </layers>
 <schematic xreflabel="%F%N/%S.%C%R" xrefpart="/%S.%C%R">
@@
 </classes>
 <parts>
-<part name="IC2-ATTINY85" library="atmel" deviceset="TINY15L" device="P"/>
+<part name="STM32F103C8" library="atmel" deviceset="TINY15L" device="P"/>
 <part name="NIXI-SOCKET" library="belton-engineering" deviceset="VT9" device="-PT"/>
 <part name="IC1" library="linear" deviceset="78*" device="T" technology="05"/>
@@
 <text x="170.18" y="45.72" size="1.9304" layer="91">HV 100-400 V</text>
 <text x="48.26" y="96.52" size="5.08" layer="91">Nixi  Test</text>
+<frame x1="-45.72" y1="-5.08" x2="193.04" y2="109.22" columns="8" rows="5" layer="116" border-left="no" border-top="no" border-right="no" border-bottom="no"/>
 </plain>
 <instances>
-<instance part="IC2-ATTINY85" gate="G$1" x="22.86" y="48.26"/>
+<instance part="STM32F103C8" gate="G$1" x="22.86" y="48.26"/>
 <instance part="NIXI-SOCKET" gate="G$1" x="152.4" y="68.58"/>
 <instance part="IC1" gate="A1" x="17.78" y="81.28"/>
@@
 <pinref part="R1" gate="G$1" pin="1"/>
 <wire x1="99.06" y1="50.8" x2="99.06" y2="45.72" width="0.1524" layer="91"/>
+<junction x="114.3" y="50.8"/>
 </segment>
 </net>
@@
 <segment>
 <pinref part="DEBUG" gate="-2" pin="S"/>
-<pinref part="IC2-ATTINY85" gate="G$1" pin="(ADC0)PB5"/>
+<pinref part="STM32F103C8" gate="G$1" pin="(ADC0)PB5"/>
 <wire x1="45.72" y1="53.34" x2="40.64" y2="53.34" width="0.1524" layer="91"/>
 </segment>
@@
 <pinref part="NIXI-SOCKET" gate="G$1" pin="8"/>
 <pinref part="NIXI-SOCKET" gate="G$1" pin="9"/>
+<junction x="149.86" y="43.18"/>
 </segment>
 </net>
 <net name="N$5" class="0">
 <segment>
-<pinref part="IC2-ATTINY85" gate="G$1" pin="(ADC1)PB2"/>
+<pinref part="STM32F103C8" gate="G$1" pin="(ADC1)PB2"/>
 <wire x1="40.64" y1="45.72" x2="48.26" y2="45.72" width="0.1524" layer="91"/>
 <wire x1="48.26" y1="45.72" x2="48.26" y2="40.64" width="0.1524" layer="91" curve="-180"/>
@@
 <net name="N$7" class="0">
 <segment>
-<pinref part="IC2-ATTINY85" gate="G$1" pin="(OCP)PB1"/>
+<pinref part="STM32F103C8" gate="G$1" pin="(OCP)PB1"/>
 <pinref part="R2" gate="G$1" pin="1"/>
 <wire x1="40.64" y1="43.18" x2="71.12" y2="43.18" width="0.1524" layer="91"/>
