File: nixi/nixi/nixiRemoteControlReceiver.sch (EAGLE design)
At the start: 16 parts, among them IC1 7805L, IC2 4081D, IC3 40106D, K1 TXD2-1.5V, K2 TXD2-1.5V, T1 2N3904, T2 2N3904

Commit message: nixi started
Parts:
- removed C1: (no value), resistor:CPOL-EUE10-20
- added R2: 100, resistor:R-EU_0411/15
- added R3: 10k, resistor:R-EU_0411/15
- C2: value (none) -> 47uF/16V
Connections:
- new net N$1: K1G$2.O, X1.B-3
- new net N$10: D1.C, K2_.+
- new net N$11: C2.+, T1.E
- new net N$12: R3.2
- new net N$13: K1_.-
- new net N$14: K1_.+
- new net N$2: X1.B-4
- new net N$3: K1G$1.O, X2.B-8
- new net N$4: K1G$1.S, X2.B-7
- new net N$5: K2_.-, T2.C
- new net N$6: R1.2, T2.B
- new net N$7: K2G$1.O, X2.B-4
- new net N$8: X2.B-5
- new net N$9: D1.A, R2.1
- net +12V: now also R2.2
- net +5V: now also IC1.VO, T1.C
- net GND: now also C2.-, R3.1, T2.E
Other:
- moved on the sheet: C2, C3, C4, D1, IC1, IC2A, IC2B, IC2C, IC2D, IC3A, IC3B, IC3C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

Commit message: nixi started
Connections:
- new net N$15: IC3A.I
- new net N$16: IC3B.I, X2.B-6
- new net N$17: IC3C.O, IC3D.I
- new net N$19: IC3E.O, T1.B
- new net N$21: IC2A.I1, IC3D.O
- new net N$22: IC2A.O, R1.1
- new net N$23: IC3F.O
- new net N$24: IC3A.O, IC3F.I
- net N$12: now also IC3C.I
Other:
- note added: "green"
- note added: "grey"
- note added: "red"
- note added: "white"
- moved on the sheet: IC3B, IC3C, IC3D, IC3E, IC3F
Changed lines of the file:
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@@
 <rectangle x1="-35.56" y1="-22.86" x2="-2.54" y2="22.86" layer="91"/>
 <text x="-33.02" y="25.4" size="2.54" layer="91">receiverboard</text>
+<text x="-27.94" y="91.44" size="2.54" layer="91">green</text>
+<text x="-17.78" y="71.12" size="2.54" layer="91">grey</text>
+<text x="106.68" y="10.16" size="2.54" layer="91">red</text>
+<text x="111.76" y="38.1" size="2.54" layer="91">white</text>
 </plain>
 <instances>
@@
 <instance part="IC2" gate="D" x="195.58" y="66.04"/>
 <instance part="IC3" gate="A" x="20.32" y="88.9"/>
-<instance part="IC3" gate="B" x="20.32" y="78.74"/>
-<instance part="IC3" gate="C" x="20.32" y="68.58"/>
-<instance part="IC3" gate="D" x="20.32" y="58.42"/>
-<instance part="IC3" gate="E" x="20.32" y="48.26"/>
-<instance part="IC3" gate="F" x="20.32" y="38.1"/>
+<instance part="IC3" gate="B" x="20.32" y="68.58"/>
+<instance part="IC3" gate="C" x="93.98" y="66.04"/>
+<instance part="IC3" gate="D" x="114.3" y="66.04"/>
+<instance part="IC3" gate="E" x="38.1" y="68.58"/>
+<instance part="IC3" gate="F" x="60.96" y="88.9"/>
 <instance part="X1" gate="G$1" x="33.02" y="-25.4" rot="R270"/>
 <instance part="X2" gate="G$1" x="162.56" y="-25.4" rot="R270"/>
@@
 </segment>
 </net>
-<net name="N$12" class="0">
-<segment>
-<pinref part="R3" gate="G$1" pin="2"/>
-<wire x1="68.58" y1="66.04" x2="86.36" y2="66.04" width="0.1524" layer="91"/>
-</segment>
-</net>
 <net name="N$13" class="0">
 <segment>
@@
 </segment>
 </net>
+<net name="N$15" class="0">
+<segment>
+<wire x1="5.08" y1="17.78" x2="10.16" y2="17.78" width="0.1524" layer="91"/>
+<wire x1="10.16" y1="17.78" x2="10.16" y2="30.48" width="0.1524" layer="91"/>
+<wire x1="10.16" y1="30.48" x2="-30.48" y2="30.48" width="0.1524" layer="91"/>
+<wire x1="-30.48" y1="30.48" x2="-30.48" y2="88.9" width="0.1524" layer="91"/>
+<pinref part="IC3" gate="A" pin="I"/>
+<wire x1="-30.48" y1="88.9" x2="10.16" y2="88.9" width="0.1524" layer="91"/>
+</segment>
+</net>
+<net name="N$16" class="0">
+<segment>
+<pinref part="X2" gate="G$1" pin="B-6"/>
+<wire x1="157.48" y1="-17.78" x2="157.48" y2="43.18" width="0.1524" layer="91"/>
+<wire x1="157.48" y1="43.18" x2="33.02" y2="43.18" width="0.1524" layer="91"/>
+<wire x1="33.02" y1="43.18" x2="33.02" y2="30.48" width="0.1524" layer="91"/>
+<wire x1="33.02" y1="30.48" x2="12.7" y2="30.48" width="0.1524" layer="91"/>
+<wire x1="12.7" y1="30.48" x2="12.7" y2="33.02" width="0.1524" layer="91"/>
+<wire x1="12.7" y1="33.02" x2="-27.94" y2="33.02" width="0.1524" layer="91"/>
+<wire x1="-27.94" y1="33.02" x2="-27.94" y2="68.58" width="0.1524" layer="91"/>
+<pinref part="IC3" gate="B" pin="I"/>
+<wire x1="-27.94" y1="68.58" x2="10.16" y2="68.58" width="0.1524" layer="91"/>
+</segment>
+</net>
+<net name="N$19" class="0">
+<segment>
+<pinref part="IC3" gate="E" pin="O"/>
+<pinref part="T1" gate="G1" pin="B"/>
+<wire x1="48.26" y1="68.58" x2="63.5" y2="68.58" width="0.1524" layer="91"/>
+</segment>
+</net>
+<net name="N$12" class="0">
+<segment>
+<pinref part="R3" gate="G$1" pin="2"/>
+<wire x1="68.58" y1="66.04" x2="83.82" y2="66.04" width="0.1524" layer="91"/>
+<pinref part="IC3" gate="C" pin="I"/>
+<wire x1="83.82" y1="66.04" x2="86.36" y2="66.04" width="0.1524" layer="91"/>
+<junction x="83.82" y="66.04"/>
+</segment>
+</net>
+<net name="N$21" class="0">
+<segment>
+<pinref part="IC2" gate="A" pin="I1"/>
+<wire x1="132.08" y1="78.74" x2="165.1" y2="78.74" width="0.1524" layer="91"/>
+<wire x1="132.08" y1="66.04" x2="132.08" y2="78.74" width="0.1524" layer="91"/>
+<pinref part="IC3" gate="D" pin="O"/>
+<wire x1="124.46" y1="66.04" x2="132.08" y2="66.04" width="0.1524" layer="91"/>
+</segment>
+</net>
+<net name="N$23" class="0">
+<segment>
+<pinref part="IC3" gate="F" pin="O"/>
+<wire x1="71.12" y1="88.9" x2="134.62" y2="88.9" width="0.1524" layer="91"/>
+<wire x1="167.64" y1="83.82" x2="167.64" y2="81.28" width="0.1524" layer="91"/>
+<wire x1="134.62" y1="83.82" x2="167.64" y2="83.82" width="0.1524" layer="91"/>
+<wire x1="134.62" y1="88.9" x2="134.62" y2="83.82" width="0.1524" layer="91"/>
+</segment>
+</net>
+<net name="N$22" class="0">
+<segment>
+<pinref part="IC2" gate="A" pin="O"/>
+<wire x1="180.34" y1="81.28" x2="182.88" y2="81.28" width="0.1524" layer="91"/>
+<pinref part="R1" gate="G$1" pin="1"/>
+<wire x1="182.88" y1="81.28" x2="182.88" y2="-2.54" width="0.1524" layer="91"/>
+</segment>
+</net>
+<net name="N$24" class="0">
+<segment>
+<pinref part="IC3" gate="A" pin="O"/>
+<wire x1="30.48" y1="88.9" x2="50.8" y2="88.9" width="0.1524" layer="91"/>
+<pinref part="IC3" gate="F" pin="I"/>
+</segment>
+</net>
+<net name="N$17" class="0">
+<segment>
+<pinref part="IC3" gate="C" pin="O"/>
+<pinref part="IC3" gate="D" pin="I"/>
+</segment>
+</net>

Commit message: reg save
Connections:
- net N$2: now also K1G$2.P
- net N$4: now also K1G$1.P; no longer K1G$1.S
- net N$7: now also K2G$1.S; no longer K2G$1.O
Other:
- note added: "(maybe not needed at all)"
- note added: "170 V pwm"
- note added: "alarm reset"
- note added: "alarm state"
- note added: "blue leds"
- note added: "prevent multiple events by delaying"
Changed lines of the file:
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@@
 <text x="106.68" y="10.16" size="2.54" layer="91">red</text>
 <text x="111.76" y="38.1" size="2.54" layer="91">white</text>
+<text x="139.7" y="45.72" size="2.54" layer="91">alarm state</text>
+<text x="165.1" y="40.64" size="2.54" layer="91">alarm reset</text>
+<text x="127" y="38.1" size="2.54" layer="91">170 V pwm</text>
+<text x="124.46" y="-7.62" size="2.54" layer="91">blue leds</text>
+<text x="73.66" y="78.74" size="1.778" layer="91">prevent multiple events by delaying</text>
+<text x="73.66" y="73.66" size="1.778" layer="91">(maybe not needed at all)</text>
 </plain>
 <instances>
@@
 <wire x1="40.64" y1="-12.7" x2="96.52" y2="-12.7" width="0.1524" layer="91"/>
 <wire x1="96.52" y1="-12.7" x2="96.52" y2="0" width="0.1524" layer="91"/>
-<wire x1="96.52" y1="0" x2="121.92" y2="0" width="0.1524" layer="91"/>
-<wire x1="121.92" y1="0" x2="121.92" y2="17.78" width="0.1524" layer="91"/>
-<wire x1="121.92" y1="17.78" x2="127" y2="17.78" width="0.1524" layer="91"/>
+<wire x1="96.52" y1="0" x2="129.54" y2="0" width="0.1524" layer="91"/>
+<pinref part="K1" gate="G$2" pin="P"/>
+<wire x1="129.54" y1="0" x2="129.54" y2="10.16" width="0.1524" layer="91"/>
 </segment>
 </net>
@@
 <net name="N$4" class="0">
 <segment>
-<pinref part="K1" gate="G$1" pin="S"/>
-<wire x1="124.46" y1="30.48" x2="121.92" y2="30.48" width="0.1524" layer="91"/>
-<wire x1="121.92" y1="30.48" x2="121.92" y2="35.56" width="0.1524" layer="91"/>
 <wire x1="121.92" y1="35.56" x2="147.32" y2="35.56" width="0.1524" layer="91"/>
 <wire x1="147.32" y1="35.56" x2="147.32" y2="-15.24" width="0.1524" layer="91"/>
@@
 <pinref part="X2" gate="G$1" pin="B-7"/>
 <wire x1="154.94" y1="-15.24" x2="154.94" y2="-17.78" width="0.1524" layer="91"/>
+<wire x1="121.92" y1="35.56" x2="121.92" y2="22.86" width="0.1524" layer="91"/>
+<pinref part="K1" gate="G$1" pin="P"/>
+<wire x1="121.92" y1="22.86" x2="129.54" y2="22.86" width="0.1524" layer="91"/>
 </segment>
 </net>
@@
 <net name="N$7" class="0">
 <segment>
-<pinref part="K2" gate="G$1" pin="O"/>
-<wire x1="175.26" y1="33.02" x2="177.8" y2="33.02" width="0.1524" layer="91"/>
-<wire x1="177.8" y1="33.02" x2="177.8" y2="-10.16" width="0.1524" layer="91"/>
+<wire x1="177.8" y1="38.1" x2="177.8" y2="-10.16" width="0.1524" layer="91"/>
 <wire x1="177.8" y1="-10.16" x2="162.56" y2="-10.16" width="0.1524" layer="91"/>
 <pinref part="X2" gate="G$1" pin="B-4"/>
 <wire x1="162.56" y1="-10.16" x2="162.56" y2="-17.78" width="0.1524" layer="91"/>
+<wire x1="177.8" y1="38.1" x2="165.1" y2="38.1" width="0.1524" layer="91"/>
+<pinref part="K2" gate="G$1" pin="S"/>
+<wire x1="165.1" y1="38.1" x2="165.1" y2="33.02" width="0.1524" layer="91"/>
 </segment>
 </net>

Commit message: reg save
Connections:
- net N$8: now also K2G$1.P
Other:
- moved on the sheet: D1, K2, R1, R2, T2
Changed lines of the file:
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@@
 <text x="111.76" y="38.1" size="2.54" layer="91">white</text>
 <text x="139.7" y="45.72" size="2.54" layer="91">alarm state</text>
-<text x="165.1" y="40.64" size="2.54" layer="91">alarm reset</text>
+<text x="165.1" y="35.56" size="2.54" layer="91">alarm reset</text>
 <text x="127" y="38.1" size="2.54" layer="91">170 V pwm</text>
 <text x="124.46" y="-7.62" size="2.54" layer="91">blue leds</text>
@@
 <instances>
 <instance part="T1" gate="G1" x="66.04" y="68.58"/>
-<instance part="T2" gate="G1" x="195.58" y="-2.54"/>
+<instance part="T2" gate="G1" x="195.58" y="15.24"/>
 <instance part="IC1" gate="A1" x="71.12" y="27.94"/>
 <instance part="C2" gate="G$1" x="68.58" y="60.96"/>
 <instance part="C3" gate="G$1" x="88.9" y="20.32"/>
-<instance part="R1" gate="G$1" x="187.96" y="-2.54"/>
-<instance part="D1" gate="1" x="198.12" y="25.4" rot="R270"/>
+<instance part="R1" gate="G$1" x="187.96" y="15.24"/>
+<instance part="D1" gate="1" x="198.12" y="40.64" rot="R270"/>
 <instance part="K1" gate="_" x="111.76" y="20.32"/>
 <instance part="K1" gate="G$1" x="129.54" y="25.4"/>
 <instance part="K1" gate="G$2" x="129.54" y="12.7"/>
-<instance part="K2" gate="_" x="198.12" y="7.62"/>
-<instance part="K2" gate="G$1" x="170.18" y="27.94"/>
+<instance part="K2" gate="_" x="198.12" y="25.4"/>
+<instance part="K2" gate="G$1" x="170.18" y="22.86"/>
 <instance part="IC2" gate="A" x="172.72" y="81.28"/>
 <instance part="IC2" gate="B" x="172.72" y="66.04"/>
@@
 <instance part="SUPPLY3" gate="GND" x="78.74" y="7.62"/>
 <instance part="C4" gate="G$1" x="58.42" y="20.32"/>
-<instance part="SUPPLY5" gate="+12V" x="198.12" y="40.64"/>
-<instance part="R2" gate="G$1" x="198.12" y="33.02" rot="R90"/>
-<instance part="SUPPLY6" gate="GND" x="198.12" y="-10.16"/>
+<instance part="SUPPLY5" gate="+12V" x="198.12" y="53.34"/>
+<instance part="R2" gate="G$1" x="198.12" y="48.26" rot="R90"/>
+<instance part="SUPPLY6" gate="GND" x="198.12" y="10.16"/>
 <instance part="SUPPLY7" gate="+5V" x="68.58" y="76.2"/>
 <instance part="R3" gate="G$1" x="86.36" y="60.96" rot="R90"/>
@@
 <pinref part="SUPPLY5" gate="+12V" pin="+12V"/>
 <pinref part="R2" gate="G$1" pin="2"/>
+<wire x1="198.12" y1="53.34" x2="198.12" y2="50.8" width="0.1524" layer="91"/>
 </segment>
 </net>
@@
 <pinref part="T2" gate="G1" pin="E"/>
 <pinref part="SUPPLY6" gate="GND" pin="GND"/>
+<wire x1="198.12" y1="12.7" x2="198.12" y2="10.16" width="0.1524" layer="91"/>
 </segment>
 <segment>
@@
 <net name="N$7" class="0">
 <segment>
-<wire x1="177.8" y1="38.1" x2="177.8" y2="-10.16" width="0.1524" layer="91"/>
-<wire x1="177.8" y1="-10.16" x2="162.56" y2="-10.16" width="0.1524" layer="91"/>
+<wire x1="180.34" y1="33.02" x2="180.34" y2="-10.16" width="0.1524" layer="91"/>
+<wire x1="180.34" y1="-10.16" x2="162.56" y2="-10.16" width="0.1524" layer="91"/>
 <pinref part="X2" gate="G$1" pin="B-4"/>
 <wire x1="162.56" y1="-10.16" x2="162.56" y2="-17.78" width="0.1524" layer="91"/>
-<wire x1="177.8" y1="38.1" x2="165.1" y2="38.1" width="0.1524" layer="91"/>
+<wire x1="180.34" y1="33.02" x2="165.1" y2="33.02" width="0.1524" layer="91"/>
 <pinref part="K2" gate="G$1" pin="S"/>
-<wire x1="165.1" y1="38.1" x2="165.1" y2="33.02" width="0.1524" layer="91"/>
+<wire x1="165.1" y1="33.02" x2="165.1" y2="27.94" width="0.1524" layer="91"/>
 </segment>
 </net>
@@
 <wire x1="160.02" y1="-7.62" x2="160.02" y2="-17.78" width="0.1524" layer="91"/>
 <wire x1="160.02" y1="-7.62" x2="170.18" y2="-7.62" width="0.1524" layer="91"/>
-<wire x1="170.18" y1="-7.62" x2="170.18" y2="27.94" width="0.1524" layer="91"/>
+<wire x1="170.18" y1="-7.62" x2="170.18" y2="20.32" width="0.1524" layer="91"/>
+<pinref part="K2" gate="G$1" pin="P"/>
+<wire x1="170.18" y1="20.32" x2="170.18" y2="22.86" width="0.1524" layer="91"/>
+<junction x="170.18" y="20.32"/>
 </segment>
 </net>
@@
 <pinref part="D1" gate="1" pin="C"/>
 <pinref part="K2" gate="_" pin="+"/>
-<wire x1="198.12" y1="22.86" x2="198.12" y2="12.7" width="0.1524" layer="91"/>
+<wire x1="198.12" y1="38.1" x2="198.12" y2="30.48" width="0.1524" layer="91"/>
 </segment>
 </net>
@@
 <wire x1="180.34" y1="81.28" x2="182.88" y2="81.28" width="0.1524" layer="91"/>
 <pinref part="R1" gate="G$1" pin="1"/>
-<wire x1="182.88" y1="81.28" x2="182.88" y2="-2.54" width="0.1524" layer="91"/>
-</segment>
-</net>
+<wire x1="182.88" y1="81.28" x2="182.88" y2="15.24" width="0.1524" layer="91"/>
+</segment>
+</net>
