File: boosterPac/boosterPac/centuryBoosterPac.sch (EAGLE design)
At the start: 5 parts, among them J1 22-05-7028-02, J2 22-05-7028-02, Q1 BSS123

Commit message: reg save
Parts:
- added 1N1, 1N539: 1N5400, diode:1N5400
- added 2901N: (no value), ic-package:DIL14
- added IC1: 317T, linear:317T
- added R10, R5, R9: 2.4k, resistor:R-EU_0309/10
- added R11: 5.1k, resistor:R-EU_0309/10
- added R12: 2M, rcl:R-TRIMM3202
- added R3: 240, resistor:R-EU_0309/10
- added R4: 300, rcl:R-TRIMM3202
- added R6: 20k, resistor:R-EU_0309/10
- added R7: 150, resistor:R-EU_0309/10
- added R8: 510, resistor:R-EU_0309/10
- R2: value 1k -> 5k
Connections:
- new net N$10: 2901N.7, R10.1, R8.2
- new net N$11: 2901N.9, R7.2, R8.1
- new net N$12: 2901N.11, R7.1
- new net N$2: 1N1.A, IC1.VO, R3.2
- new net N$3: R4.A, R5.1
- new net N$4: IC1.ADJ, R3.1, R4.S
- new net N$5: R11.1, R5.2
- new net N$6: R11.2, R6.1
- new net N$7: R12.A, R6.2
- new net N$8: R12.S
- new net N$9: R10.2, R9.2
- net +15V: now also 1N539.A, 1N539.C, IC1.VI
- net GND: now also 1N1.C, R12.E, R9.1
Other:
- note added: "======"
- note added: "power from power adapter"
- note removed: "power form lima"
- moved on the sheet: J1-1, J1-2, J2-1, J2-2, Q1, R1, R2

Commit message: reg save
Parts:
- removed R10: 2.4k, resistor:R-EU_0309/10
- added 46A837: 1N5400, diode:1N5400
- added LED1_YEL, LED2_RED, LED3_RED, LED6_RED, LED7_GRN: (no value), led:LED
- added R13: 10k, resistor:R-EU_0309/10
- added R14: 210, resistor:R-EU_0309/10
- added R15, R16, R17, R18, R20: 1k, resistor:R-EU_0309/10
- added R19: 430, resistor:R-EU_0309/10
- R9: value 2.4k -> 1k
Connections:
- removed net N$10: 2901N.7, R10.1, R8.2
- new net N$14: 2901N.5, 46A837.C, R14.1, R19.2, R9.2
- new net N$15: LED6_RED.C, R16.1
- new net N$16: LED3_RED.C, R17.1
- new net N$17: LED2_RED.C, R18.1
- new net N$18: LED1_YEL.C, R20.1
- new net N$20: R18.2
- new net N$21: R17.2
- new net N$22: R16.2
- new net N$23: 2901N.13, LED2_RED.A
- new net N$24: 2901N.14, LED3_RED.A
- new net N$25: 2901N.1, LED6_RED.A
- new net N$26: 2901N.2, LED7_GRN.A
- new net N$27: 2901N.7, R19.1, R8.2
- net GND: now also R14.2, R15.2, R20.2
- net N$5: now also 2901N.12, 46A837.A, LED1_YEL.A, R13.1
- net N$9: now also LED7_GRN.C, R15.1; no longer R10.2, R9.2
Other:
- moved on the sheet: 2901N, R7, R8, R9

Commit message: reg save
Parts:
- added D6: 1N5400, diode:1N5400
- R12: value 2M -> 500
- renumbered 1N1 to 1N539-
Connections:
- net +15V renamed N$10
- removed net N$7: R12.A, R6.2
- new net N$28: 1N539-.C, D6.C, R12.A, R12.S, R14.2, R9.1
- new net N$6: R11.1, R5.1
- net GND: no longer 1N539-.C, R12.E, R14.2, R9.1
- net N$3: now also R5.2; no longer R5.1
- net N$5: no longer R11.1, R5.2
- net N$8: now also R12.E, R6.2; no longer R12.S
Other:
- moved on the sheet: R11, R12, R18, R20, R5, R6

Commit message: reg save
Parts:
- removed D6: 1N5400, diode:1N5400
- removed R18, R20: 1k, resistor:R-EU_0309/10
- removed R19: 430, resistor:R-EU_0309/10
- added 46A837-D8, X-D6: 1N5400, diode:1N5400
- added R10: 150, resistor:R-EU_0309/10
- added VR1: 300, rcl:R-TRIMM3202
- added VR2: 5K, rcl:R-TRIMM3202
- R11: value 5.1k -> 430
- R12: value 500 -> 510; device rcl:R-TRIMM3202 -> resistor:R-EU_0309/10
- R13: value 10k -> 5.1k
- R14: value 210 -> 20k
- R16: value 1k -> 5k
- R2: value 5k -> 1k
- R3: value 240 -> 1k
- R4: value 300 -> 1k; device rcl:R-TRIMM3202 -> resistor:R-EU_0309/10
- R5: value 2.4k -> 1k
- R6: value 20k -> 210
- R7: value 150 -> 240
- R8: value 510 -> 2.4k
- R9: value 1k -> 10k
- renumbered 1N539 to 1N539-D9, 1N539- to 1N539-D7, 46A837 to 46A837-D10, LED6_RED to LED4_RED, LED7_GRN to LED5_GRN
Connections:
- removed net GND1: J2-2.S, Q1.D
- removed net N$28: 1N539-D7.C, D6.C, R12.A, R12.S, R14.2, R9.1
- removed net N$6: R11.1, R5.1
- new net +UB: 1N539-D7.C, 46A837-D8.C, R15.1, R6.2, VR2.A, VR2.S
- new net -UB: 46A837-D8.A, J1-2.S, J2-1.S, Q1.S, R16.1
- new net FZ: J2-2.S, Q1.D, R13.1, R8.1, R9.2, X-D6.A
- net GND: now also R1.2, R5.2; no longer J1-2.S, J2-1.S, Q1.S, R15.2, R2.1, R20.2
- net N$1: now also R16.2, R17.1; no longer R1.1, R2.2
- net N$10: now also R17.2; no longer R1.2
- net N$11: now also R10.2, R12.1; no longer R7.2, R8.1
- net N$12: now also R10.1; no longer R7.1
- net N$14: now also R11.1, R15.2, R6.1; no longer R14.1, R19.2, R9.2
- net N$15: now also R4.1; no longer R16.1
- net N$16: now also R3.1; no longer R17.1
- net N$17: now also R2.1; no longer R18.1
- net N$18: now also R1.1; no longer R20.1
- net N$19: now also 2901N.6, R13.2, R14.1; no longer R11.2, R6.1
- net N$2: now also R7.2; no longer R3.2
- net N$20: now also R2.2; no longer R18.2
- net N$21: now also R3.2; no longer R17.2
- net N$22: now also R4.2; no longer R16.2
- net N$27: now also R11.2, R12.2; no longer R19.1, R8.2
- net N$3: now also R8.2, VR1.A; no longer R4.A, R5.2
- net N$4: now also R7.1, VR1.S; no longer R3.1, R4.S
- net N$5: now also R9.1; no longer R13.1
- net N$8: now also R14.2, VR2.E; no longer R12.E, R6.2
- net N$9: now also R5.1; no longer R15.1
Other:
- note added: "entry 12V car adapter"
- note added: "power from 220V power adapter"
- note removed: "exit to accu"
- note removed: "power from power adapter"
- moved on the sheet: R1, R11, R13, R14, R15, R16, R17, R2, R3, R5, R6, R7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

Commit message: reg save
Connections:
- removed net GND: R1.2, R5.2
- removed net N$26: 2901N.2, LED5_GRN.A
- new net N$6: 2901N.2, LED5_GRN.A, LED5_GRN.C, R5.1
- net +UB: now also R1.2, R5.2
- net N$14: no longer 46A837-D10.C, R11.1, R15.2, R6.1
- net N$15: no longer LED4_RED.C
- net N$16: no longer LED3_RED.C
- net N$17: now also LED2_RED.A; no longer LED2_RED.C
- net N$18: now also LED1_YEL.A; no longer LED1_YEL.C
- net N$23: now also LED2_RED.C; no longer LED2_RED.A
- net N$24: now also LED3_RED.C; no longer LED3_RED.A
- net N$25: now also LED4_RED.C; no longer LED4_RED.A
- net N$5: now also LED1_YEL.C; no longer LED1_YEL.A
- net N$9: now also 2901N.3, 46A837-D10.C, R11.1, R15.2, R6.1; no longer LED5_GRN.C, R5.1
Other:
- note added: "push button"
- note removed: "entry 12V car adapter"
- moved on the sheet: LED1_YEL, LED2_RED, LED3_RED, LED4_RED, LED5_GRN

Commit message: reg save
Parts:
- added BATTERY: 22-05-7028-02, con-molex:22-05-7028-02
- added R18: xk?, resistor:R-EU_0309/10
- added S1: 5501-1LED, switch:5501-1LED
Connections:
- removed net -UB: 46A837-D8.A, J1-2.S, J2-1.S, Q1.S, R16.1
- removed net FZ: J2-2.S, Q1.D, R13.1, R8.1, R9.2, X-D6.A
- removed net N$5: 2901N.12, 46A837-D10.A, LED1_YEL.C, R9.1
- new net GND: 46A837-D8.A, BATTERY-2.S, J1-2.S, J2-1.S, Q1.S, R16.1
- new net N$26: R18.1
- new net N$28: R18.2, S1-1.NO
- new net UVAR-1: 2901N.12, 46A837-D10.A, J2-2.S, LED1_YEL.C, Q1.D, R13.1, R8.1, R9.2, X-D6.A
- net +UB: now also BATTERY-1.S
Other:
- note added: "load simulation for battery test on leds ???"
- note added: "protection ?"
- moved on the sheet: R9

Commit message: reg save
Parts:
- removed 1N539-D9, 46A837-D8: 1N5400, diode:1N5400
- added D8, D9: 1N5400, diode:1N5400
- added J4: 22-05-7028-02, con-molex:22-05-7028-02
- renumbered 46A837-D10 to D10, X-D6 to D6
Connections:
- new net -UB: J2-1.S
- new net N$29: IC1.VI
- net +UB: now also D8.C; no longer 46A837-D8.C
- net GND: now also D8.A; no longer 46A837-D8.A, J2-1.S, Q1.S
- net N$10: no longer 1N539-D9.A, 1N539-D9.C, IC1.VI
- net N$16: now also LED3_RED.A
Other:
- note added: "?"
Changed lines of the file:
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@@
 <part name="R16" library="resistor" deviceset="R-EU_" device="0309/10" value="5k"/>
 <part name="J2" library="con-molex" deviceset="22-?-02" device="05-7028"/>
-<part name="1N539-D9" library="diode" deviceset="1N5400" device=""/>
+<part name="D9" library="diode" deviceset="1N5400" device=""/>
 <part name="IC1" library="linear" deviceset="*317" device="T"/>
 <part name="1N539-D7" library="diode" deviceset="1N5400" device=""/>
@@
 <part name="2901N" library="ic-package" deviceset="DIL14" device=""/>
 <part name="R9" library="resistor" deviceset="R-EU_" device="0309/10" value="10k"/>
-<part name="46A837-D10" library="diode" deviceset="1N5400" device=""/>
+<part name="D10" library="diode" deviceset="1N5400" device=""/>
 <part name="R6" library="resistor" deviceset="R-EU_" device="0309/10" value="210"/>
 <part name="LED1_YEL" library="led" deviceset="LED" device=""/>
@@
 <part name="SUPPLY3" library="supply2" deviceset="-UB" device=""/>
 <part name="R11" library="resistor" deviceset="R-EU_" device="0309/10" value="430"/>
-<part name="X-D6" library="diode" deviceset="1N5400" device=""/>
-<part name="46A837-D8" library="diode" deviceset="1N5400" device=""/>
+<part name="D6" library="diode" deviceset="1N5400" device=""/>
+<part name="D8" library="diode" deviceset="1N5400" device=""/>
 <part name="SUPPLY5" library="supply2" deviceset="+UB" device=""/>
 <part name="SUPPLY4" library="supply2" deviceset="+UB" device=""/>
@@
 <part name="SUPPLY8" library="supply2" deviceset="GND" device=""/>
 <part name="R18" library="resistor" deviceset="R-EU_" device="0309/10" value="xk?"/>
+<part name="J4" library="con-molex" deviceset="22-?-02" device="05-7028"/>
 </parts>
 <sheets>
@@
 <plain>
 <text x="-78.74" y="106.68" size="1.778" layer="91">power from 220V power adapter</text>
-<text x="-10.16" y="137.16" size="1.778" layer="91">======</text>
-<text x="-10.16" y="137.16" size="1.778" layer="91">======</text>
+<text x="-7.62" y="137.16" size="1.778" layer="91">======</text>
 <text x="35.56" y="132.08" size="1.778" layer="91" rot="R270">======</text>
 <text x="119.38" y="96.52" size="1.778" layer="91" rot="R270">======</text>
@@
 <text x="20.32" y="78.74" size="1.778" layer="91">load simulation for battery test on leds ???</text>
 <text x="-58.42" y="58.42" size="1.778" layer="91">protection ?</text>
+<text x="-33.02" y="35.56" size="3.81" layer="91">?</text>
 </plain>
 <instances>
 <instance part="J1" gate="-1" x="-50.8" y="104.14" rot="R180"/>
 <instance part="J1" gate="-2" x="-50.8" y="99.06" rot="R180"/>
-<instance part="SUPPLY2" gate="GND" x="-40.64" y="35.56"/>
+<instance part="SUPPLY2" gate="GND" x="-38.1" y="35.56"/>
 <instance part="Q1" gate="G$1" x="-27.94" y="60.96"/>
 <instance part="R17" gate="G$1" x="-38.1" y="63.5" rot="R90"/>
@@
 <instance part="J2" gate="-1" x="17.78" y="63.5" rot="R90"/>
 <instance part="J2" gate="-2" x="12.7" y="63.5" rot="R90"/>
-<instance part="1N539-D9" gate="1" x="-12.7" y="139.7"/>
+<instance part="D9" gate="1" x="-10.16" y="139.7"/>
 <instance part="IC1" gate="A1" x="17.78" y="137.16"/>
 <instance part="1N539-D7" gate="1" x="38.1" y="134.62" rot="R270"/>
@@
 <instance part="2901N" gate="G$1" x="88.9" y="58.42" rot="R90"/>
 <instance part="R9" gate="G$1" x="-10.16" y="96.52" rot="R180"/>
-<instance part="46A837-D10" gate="1" x="121.92" y="99.06" rot="R270"/>
+<instance part="D10" gate="1" x="121.92" y="99.06" rot="R270"/>
 <instance part="R6" gate="G$1" x="121.92" y="27.94" rot="R270"/>
 <instance part="LED1_YEL" gate="G$1" x="48.26" y="66.04" rot="R90"/>
@@
 <instance part="SUPPLY3" gate="G$1" x="-25.4" y="35.56"/>
 <instance part="R11" gate="G$1" x="99.06" y="40.64"/>
-<instance part="X-D6" gate="1" x="86.36" y="7.62" rot="R90"/>
-<instance part="46A837-D8" gate="1" x="-55.88" y="63.5" rot="R180"/>
+<instance part="D6" gate="1" x="86.36" y="7.62" rot="R90"/>
+<instance part="D8" gate="1" x="-53.34" y="63.5" rot="R180"/>
 <instance part="SUPPLY5" gate="G$1" x="-71.12" y="66.04"/>
 <instance part="SUPPLY4" gate="G$1" x="30.48" y="-10.16" rot="R180"/>
@@
 <instance part="SUPPLY8" gate="GND" x="-55.88" y="76.2"/>
 <instance part="R18" gate="G$1" x="10.16" y="81.28" rot="R90"/>
+<instance part="J4" gate="-1" x="154.94" y="106.68"/>
+<instance part="J4" gate="-2" x="154.94" y="101.6"/>
 </instances>
 <busses>
@@
 <wire x1="119.38" y1="91.44" x2="121.92" y2="91.44" width="0.1524" layer="91"/>
 <wire x1="121.92" y1="91.44" x2="121.92" y2="35.56" width="0.1524" layer="91"/>
-<pinref part="46A837-D10" gate="1" pin="C"/>
+<pinref part="D10" gate="1" pin="C"/>
 <wire x1="121.92" y1="96.52" x2="121.92" y2="91.44" width="0.1524" layer="91"/>
 <pinref part="R6" gate="G$1" pin="1"/>
@@
 <wire x1="33.02" y1="45.72" x2="33.02" y2="12.7" width="0.1524" layer="91"/>
 <pinref part="R3" gate="G$1" pin="1"/>
-<wire x1="33.02" y1="45.72" x2="48.26" y2="45.72" width="0.1524" layer="91"/>
+<wire x1="33.02" y1="45.72" x2="45.72" y2="45.72" width="0.1524" layer="91"/>
+<pinref part="LED3_RED" gate="G$1" pin="A"/>
 </segment>
 </net>
@@
 <wire x1="-38.1" y1="116.84" x2="-20.32" y2="116.84" width="0.1524" layer="91"/>
 <wire x1="-20.32" y1="116.84" x2="-20.32" y2="139.7" width="0.1524" layer="91"/>
-<pinref part="1N539-D9" gate="1" pin="A"/>
 <wire x1="-20.32" y1="139.7" x2="-15.24" y2="139.7" width="0.1524" layer="91"/>
-<pinref part="1N539-D9" gate="1" pin="C"/>
-<wire x1="-15.24" y1="139.7" x2="-10.16" y2="139.7" width="0.1524" layer="91"/>
-<pinref part="IC1" gate="A1" pin="VI"/>
-<wire x1="-10.16" y1="139.7" x2="7.62" y2="139.7" width="0.1524" layer="91"/>
 </segment>
 </net>
@@
 <wire x1="22.86" y1="-7.62" x2="-5.08" y2="-7.62" width="0.1524" layer="91"/>
 <wire x1="-10.16" y1="-7.62" x2="-5.08" y2="-7.62" width="0.1524" layer="91" curve="-180"/>
-<pinref part="46A837-D8" gate="1" pin="C"/>
-<wire x1="-58.42" y1="63.5" x2="-63.5" y2="63.5" width="0.1524" layer="91"/>
+<pinref part="D8" gate="1" pin="C"/>
+<wire x1="-55.88" y1="63.5" x2="-63.5" y2="63.5" width="0.1524" layer="91"/>
 <wire x1="-63.5" y1="63.5" x2="-71.12" y2="63.5" width="0.1524" layer="91"/>
 <wire x1="-71.12" y1="63.5" x2="-71.12" y2="68.58" width="0.1524" layer="91"/>
@@
 <wire x1="-7.62" y1="40.64" x2="-7.62" y2="66.04" width="0.1524" layer="91"/>
 <wire x1="-7.62" y1="35.56" x2="-7.62" y2="40.64" width="0.1524" layer="91" curve="180"/>
-<pinref part="X-D6" gate="1" pin="A"/>
+<pinref part="D6" gate="1" pin="A"/>
 <wire x1="86.36" y1="5.08" x2="86.36" y2="-17.78" width="0.1524" layer="91"/>
 <wire x1="86.36" y1="-17.78" x2="-7.62" y2="-17.78" width="0.1524" layer="91"/>
 <wire x1="-7.62" y1="-17.78" x2="-7.62" y2="35.56" width="0.1524" layer="91"/>
-<pinref part="46A837-D10" gate="1" pin="A"/>
+<pinref part="D10" gate="1" pin="A"/>
 <wire x1="121.92" y1="109.22" x2="121.92" y2="101.6" width="0.1524" layer="91"/>
 <wire x1="25.4" y1="109.22" x2="86.36" y2="109.22" width="0.1524" layer="91"/>
@@
 <net name="GND" class="0">
 <segment>
-<pinref part="J2" gate="-1" pin="S"/>
-<wire x1="17.78" y1="38.1" x2="17.78" y2="60.96" width="0.1524" layer="91"/>
-<wire x1="-25.4" y1="38.1" x2="17.78" y2="38.1" width="0.1524" layer="91"/>
-<pinref part="SUPPLY3" gate="G$1" pin="-UB"/>
-<junction x="-25.4" y="38.1"/>
-<pinref part="Q1" gate="G$1" pin="S"/>
-<wire x1="-27.94" y1="55.88" x2="-27.94" y2="38.1" width="0.1524" layer="91"/>
-<wire x1="-27.94" y1="38.1" x2="-25.4" y2="38.1" width="0.1524" layer="91"/>
-<wire x1="-38.1" y1="38.1" x2="-27.94" y2="38.1" width="0.1524" layer="91"/>
 <pinref part="R16" gate="G$1" pin="1"/>
 <wire x1="-38.1" y1="43.18" x2="-38.1" y2="38.1" width="0.1524" layer="91"/>
 <pinref part="SUPPLY2" gate="GND" pin="GND"/>
-<pinref part="46A837-D8" gate="1" pin="A"/>
+<pinref part="D8" gate="1" pin="A"/>
 <pinref part="J1" gate="-2" pin="S"/>
 <wire x1="-48.26" y1="99.06" x2="-45.72" y2="99.06" width="0.1524" layer="91"/>
 <wire x1="-45.72" y1="99.06" x2="-45.72" y2="78.74" width="0.1524" layer="91"/>
 <wire x1="-45.72" y1="78.74" x2="-45.72" y2="63.5" width="0.1524" layer="91"/>
-<wire x1="-45.72" y1="63.5" x2="-53.34" y2="63.5" width="0.1524" layer="91"/>
+<wire x1="-45.72" y1="63.5" x2="-50.8" y2="63.5" width="0.1524" layer="91"/>
 <wire x1="-45.72" y1="63.5" x2="-45.72" y2="38.1" width="0.1524" layer="91"/>
-<wire x1="-45.72" y1="38.1" x2="-40.64" y2="38.1" width="0.1524" layer="91"/>
-<wire x1="-40.64" y1="38.1" x2="-38.1" y2="38.1" width="0.1524" layer="91"/>
+<wire x1="-45.72" y1="38.1" x2="-38.1" y2="38.1" width="0.1524" layer="91"/>
 <pinref part="BATTERY" gate="-2" pin="S"/>
 <wire x1="-71.12" y1="78.74" x2="-55.88" y2="78.74" width="0.1524" layer="91"/>
@@
 <junction x="-55.88" y="78.74"/>
 <label x="-63.5" y="78.74" size="1.778" layer="95"/>
+<wire x1="-25.4" y1="38.1" x2="-38.1" y2="38.1" width="0.1524" layer="91" style="shortdash"/>
 </segment>
 </net>
@@
 </segment>
 </net>
+<net name="-UB" class="0">
+<segment>
+<pinref part="J2" gate="-1" pin="S"/>
+<wire x1="17.78" y1="38.1" x2="17.78" y2="60.96" width="0.1524" layer="91"/>
+<wire x1="-25.4" y1="38.1" x2="17.78" y2="38.1" width="0.1524" layer="91"/>
+<pinref part="SUPPLY3" gate="G$1" pin="-UB"/>
+</segment>
+</net>
+<net name="N$29" class="0">
+<segment>
+<pinref part="IC1" gate="A1" pin="VI"/>
+<wire x1="-2.54" y1="139.7" x2="7.62" y2="139.7" width="0.1524" layer="91"/>
+</segment>
+</net>
