File: boosterPac/boosterPac/centuryBoosterPac.sch (EAGLE design)
At the start: 38 parts, among them IC1 317T, J1 22-05-7028-02, J2 22-05-7028-02, J4 22-05-7028-02, Q1 BSS123

Commit message: reg save
Connections:
- removed net -UB: J2-1.S
- removed net N$10: J1-1.S, R17.2
- new net +15V: D8.C, J1-1.S, R17.2
- net +UB: no longer D8.C
- net GND: now also J2-1.S
Other:
- note removed: "?"
- note removed: "protection ?"
- moved on the sheet: BATTERY-1, BATTERY-2, D8, J1-1, J1-2
Changed lines of the file:
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@@
 <parts>
 <part name="J1" library="con-molex" deviceset="22-?-02" device="05-7028"/>
-<part name="SUPPLY2" library="supply2" deviceset="GND" device=""/>
 <part name="Q1" library="transistor-small-signal" deviceset="BSS123" device=""/>
 <part name="R17" library="resistor" deviceset="R-EU_" device="0309/10" value="1k"/>
@@
 <part name="R18" library="resistor" deviceset="R-EU_" device="0309/10" value="xk?"/>
 <part name="J4" library="con-molex" deviceset="22-?-02" device="05-7028"/>
+<part name="SUPPLY2" library="supply2" deviceset="-UB" device=""/>
+<part name="SUPPLY9" library="supply2" deviceset="+15V" device=""/>
 </parts>
 <sheets>
@@
 <text x="20.32" y="73.66" size="1.778" layer="91">push button</text>
 <text x="20.32" y="78.74" size="1.778" layer="91">load simulation for battery test on leds ???</text>
-<text x="-58.42" y="58.42" size="1.778" layer="91">protection ?</text>
-<text x="-33.02" y="35.56" size="3.81" layer="91">?</text>
 </plain>
 <instances>
-<instance part="J1" gate="-1" x="-50.8" y="104.14" rot="R180"/>
-<instance part="J1" gate="-2" x="-50.8" y="99.06" rot="R180"/>
-<instance part="SUPPLY2" gate="GND" x="-38.1" y="35.56"/>
+<instance part="J1" gate="-1" x="-55.88" y="104.14" rot="R180"/>
+<instance part="J1" gate="-2" x="-55.88" y="93.98" rot="R180"/>
 <instance part="Q1" gate="G$1" x="-27.94" y="60.96"/>
 <instance part="R17" gate="G$1" x="-38.1" y="63.5" rot="R90"/>
@@
 <instance part="R11" gate="G$1" x="99.06" y="40.64"/>
 <instance part="D6" gate="1" x="86.36" y="7.62" rot="R90"/>
-<instance part="D8" gate="1" x="-53.34" y="63.5" rot="R180"/>
-<instance part="SUPPLY5" gate="G$1" x="-71.12" y="66.04"/>
+<instance part="D8" gate="1" x="-45.72" y="88.9"/>
+<instance part="SUPPLY5" gate="G$1" x="-71.12" y="10.16"/>
 <instance part="SUPPLY4" gate="G$1" x="30.48" y="-10.16" rot="R180"/>
 <instance part="SUPPLY6" gate="G$1" x="132.08" y="20.32"/>
 <instance part="S1" gate="-1" x="15.24" y="96.52" rot="MR0"/>
-<instance part="BATTERY" gate="-1" x="-73.66" y="63.5" rot="R180"/>
-<instance part="BATTERY" gate="-2" x="-73.66" y="78.74" rot="R180"/>
-<instance part="SUPPLY7" gate="G$1" x="-71.12" y="81.28" rot="R180"/>
-<instance part="SUPPLY8" gate="GND" x="-55.88" y="76.2"/>
+<instance part="BATTERY" gate="-1" x="-73.66" y="7.62" rot="R180"/>
+<instance part="BATTERY" gate="-2" x="-73.66" y="38.1" rot="R180"/>
+<instance part="SUPPLY7" gate="G$1" x="-71.12" y="40.64" rot="R180"/>
+<instance part="SUPPLY8" gate="GND" x="-55.88" y="35.56"/>
 <instance part="R18" gate="G$1" x="10.16" y="81.28" rot="R90"/>
 <instance part="J4" gate="-1" x="154.94" y="106.68"/>
 <instance part="J4" gate="-2" x="154.94" y="101.6"/>
+<instance part="SUPPLY2" gate="G$1" x="-55.88" y="78.74" rot="R270"/>
+<instance part="SUPPLY9" gate="+15V" x="-35.56" y="119.38"/>
 </instances>
 <busses>
@@
 <pinref part="VR2" gate="G$1" pin="E"/>
 <pinref part="R14" gate="G$1" pin="2"/>
-</segment>
-</net>
-<net name="N$10" class="0">
-<segment>
-<pinref part="J1" gate="-1" pin="S"/>
-<wire x1="-48.26" y1="104.14" x2="-43.18" y2="104.14" width="0.1524" layer="91"/>
-<wire x1="-43.18" y1="104.14" x2="-43.18" y2="116.84" width="0.1524" layer="91"/>
-<wire x1="-43.18" y1="116.84" x2="-38.1" y2="116.84" width="0.1524" layer="91"/>
-<pinref part="R17" gate="G$1" pin="2"/>
-<wire x1="-38.1" y1="116.84" x2="-38.1" y2="68.58" width="0.1524" layer="91"/>
-<wire x1="-38.1" y1="116.84" x2="-20.32" y2="116.84" width="0.1524" layer="91"/>
-<wire x1="-20.32" y1="116.84" x2="-20.32" y2="139.7" width="0.1524" layer="91"/>
-<wire x1="-20.32" y1="139.7" x2="-15.24" y2="139.7" width="0.1524" layer="91"/>
 </segment>
 </net>
@@
 <wire x1="22.86" y1="-7.62" x2="-5.08" y2="-7.62" width="0.1524" layer="91"/>
 <wire x1="-10.16" y1="-7.62" x2="-5.08" y2="-7.62" width="0.1524" layer="91" curve="-180"/>
-<pinref part="D8" gate="1" pin="C"/>
-<wire x1="-55.88" y1="63.5" x2="-63.5" y2="63.5" width="0.1524" layer="91"/>
-<wire x1="-63.5" y1="63.5" x2="-71.12" y2="63.5" width="0.1524" layer="91"/>
-<wire x1="-71.12" y1="63.5" x2="-71.12" y2="68.58" width="0.1524" layer="91"/>
+<wire x1="-63.5" y1="7.62" x2="-71.12" y2="7.62" width="0.1524" layer="91"/>
+<wire x1="-71.12" y1="7.62" x2="-71.12" y2="12.7" width="0.1524" layer="91"/>
 <pinref part="SUPPLY5" gate="G$1" pin="+UB"/>
-<junction x="-71.12" y="63.5"/>
-<wire x1="-63.5" y1="-7.62" x2="-63.5" y2="63.5" width="0.1524" layer="91"/>
+<junction x="-71.12" y="7.62"/>
+<wire x1="-63.5" y1="-7.62" x2="-63.5" y2="7.62" width="0.1524" layer="91"/>
 <pinref part="BATTERY" gate="-1" pin="S"/>
 <label x="-55.88" y="-7.62" size="1.778" layer="95"/>
@@
 <net name="GND" class="0">
 <segment>
-<pinref part="R16" gate="G$1" pin="1"/>
-<wire x1="-38.1" y1="43.18" x2="-38.1" y2="38.1" width="0.1524" layer="91"/>
-<pinref part="SUPPLY2" gate="GND" pin="GND"/>
-<pinref part="D8" gate="1" pin="A"/>
-<pinref part="J1" gate="-2" pin="S"/>
-<wire x1="-48.26" y1="99.06" x2="-45.72" y2="99.06" width="0.1524" layer="91"/>
-<wire x1="-45.72" y1="99.06" x2="-45.72" y2="78.74" width="0.1524" layer="91"/>
-<wire x1="-45.72" y1="78.74" x2="-45.72" y2="63.5" width="0.1524" layer="91"/>
-<wire x1="-45.72" y1="63.5" x2="-50.8" y2="63.5" width="0.1524" layer="91"/>
-<wire x1="-45.72" y1="63.5" x2="-45.72" y2="38.1" width="0.1524" layer="91"/>
-<wire x1="-45.72" y1="38.1" x2="-38.1" y2="38.1" width="0.1524" layer="91"/>
+<pinref part="SUPPLY8" gate="GND" pin="GND"/>
+<junction x="-60.96" y="38.1"/>
 <pinref part="BATTERY" gate="-2" pin="S"/>
-<wire x1="-71.12" y1="78.74" x2="-55.88" y2="78.74" width="0.1524" layer="91"/>
+<wire x1="-71.12" y1="38.1" x2="-55.88" y2="38.1" width="0.1524" layer="91"/>
 <pinref part="SUPPLY7" gate="G$1" pin="-UB"/>
-<junction x="-71.12" y="78.74"/>
-<pinref part="SUPPLY8" gate="GND" pin="GND"/>
-<wire x1="-55.88" y1="78.74" x2="-45.72" y2="78.74" width="0.1524" layer="91"/>
-<junction x="-55.88" y="78.74"/>
-<label x="-63.5" y="78.74" size="1.778" layer="95"/>
-<wire x1="-25.4" y1="38.1" x2="-38.1" y2="38.1" width="0.1524" layer="91" style="shortdash"/>
-</segment>
-</net>
-<net name="N$5" class="0">
-<segment>
-<wire x1="17.78" y1="63.5" x2="17.78" y2="93.98" width="0.1524" layer="91"/>
-</segment>
-</net>
-<net name="N$28" class="0">
-<segment>
-<pinref part="R18" gate="G$1" pin="2"/>
-<pinref part="S1" gate="-1" pin="NO"/>
-<wire x1="10.16" y1="86.36" x2="10.16" y2="93.98" width="0.1524" layer="91"/>
-</segment>
-</net>
-<net name="-UB" class="0">
-<segment>
+<junction x="-71.12" y="38.1"/>
+<label x="-63.5" y="38.1" size="1.778" layer="95"/>
 <pinref part="J2" gate="-1" pin="S"/>
 <wire x1="17.78" y1="38.1" x2="17.78" y2="60.96" width="0.1524" layer="91"/>
 <wire x1="-25.4" y1="38.1" x2="17.78" y2="38.1" width="0.1524" layer="91"/>
 <pinref part="SUPPLY3" gate="G$1" pin="-UB"/>
+<wire x1="-55.88" y1="38.1" x2="-53.34" y2="38.1" width="0.1524" layer="91"/>
+<pinref part="R16" gate="G$1" pin="1"/>
+<wire x1="-53.34" y1="38.1" x2="-38.1" y2="38.1" width="0.1524" layer="91"/>
+<wire x1="-38.1" y1="38.1" x2="-25.4" y2="38.1" width="0.1524" layer="91"/>
+<wire x1="-38.1" y1="43.18" x2="-38.1" y2="38.1" width="0.1524" layer="91"/>
+<junction x="-38.1" y="38.1"/>
+<pinref part="J1" gate="-2" pin="S"/>
+<wire x1="-53.34" y1="38.1" x2="-53.34" y2="78.74" width="0.1524" layer="91"/>
+<pinref part="SUPPLY2" gate="G$1" pin="-UB"/>
+<wire x1="-53.34" y1="78.74" x2="-53.34" y2="88.9" width="0.1524" layer="91"/>
+<junction x="-53.34" y="78.74"/>
+<pinref part="D8" gate="1" pin="A"/>
+<wire x1="-53.34" y1="88.9" x2="-53.34" y2="93.98" width="0.1524" layer="91"/>
+<wire x1="-48.26" y1="88.9" x2="-53.34" y2="88.9" width="0.1524" layer="91"/>
+</segment>
+</net>
+<net name="N$5" class="0">
+<segment>
+<wire x1="17.78" y1="63.5" x2="17.78" y2="93.98" width="0.1524" layer="91"/>
+</segment>
+</net>
+<net name="N$28" class="0">
+<segment>
+<pinref part="R18" gate="G$1" pin="2"/>
+<pinref part="S1" gate="-1" pin="NO"/>
+<wire x1="10.16" y1="86.36" x2="10.16" y2="93.98" width="0.1524" layer="91"/>
 </segment>
 </net>
@@
 <segment>
 <pinref part="IC1" gate="A1" pin="VI"/>
-<wire x1="-2.54" y1="139.7" x2="7.62" y2="139.7" width="0.1524" layer="91"/>
-</segment>
-</net>
+<wire x1="-7.62" y1="139.7" x2="7.62" y2="139.7" width="0.1524" layer="91"/>
+</segment>
+</net>
+<net name="+15V" class="0">
+<segment>
+<pinref part="J1" gate="-1" pin="S"/>
+<pinref part="R17" gate="G$1" pin="2"/>
+<wire x1="-38.1" y1="116.84" x2="-38.1" y2="104.14" width="0.1524" layer="91"/>
+<wire x1="-38.1" y1="104.14" x2="-38.1" y2="88.9" width="0.1524" layer="91"/>
+<wire x1="-38.1" y1="88.9" x2="-38.1" y2="68.58" width="0.1524" layer="91"/>
+<wire x1="-38.1" y1="116.84" x2="-35.56" y2="116.84" width="0.1524" layer="91"/>
+<wire x1="-35.56" y1="116.84" x2="-20.32" y2="116.84" width="0.1524" layer="91"/>
+<wire x1="-20.32" y1="116.84" x2="-20.32" y2="139.7" width="0.1524" layer="91"/>
+<wire x1="-20.32" y1="139.7" x2="-12.7" y2="139.7" width="0.1524" layer="91"/>
+<wire x1="-53.34" y1="104.14" x2="-38.1" y2="104.14" width="0.1524" layer="91"/>
+<pinref part="SUPPLY9" gate="+15V" pin="+15V"/>
+<junction x="-35.56" y="116.84"/>
+<pinref part="D8" gate="1" pin="C"/>
+<wire x1="-43.18" y1="88.9" x2="-38.1" y2="88.9" width="0.1524" layer="91"/>
+</segment>
+</net>
