File: boosterPac/boosterPac/centuryBoosterPac.sch (EAGLE design)
At the start: 37 parts, among them IC1 317T, J1 22-05-7028-02, J2 22-05-7028-02, Q1 BSS123

Commit message: reg save
Connections:
- net N$15: now also LED2_RED.A
- net N$3: no longer R8.1
- net UVAR-1: now also R9.1
Other:
- moved on the sheet: 1N539-D7, 2901N, D10, D6, D9, IC1, J2-1, J2-2, LED1_GRN, LED2_RED, LED3_RED, LED4_RED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

Commit message: reg save
Other:
- note added: "220V power adapter connected with matching adapter, S2 pressed (Uvar1 exactly 0): --- Uvar on gnd because Q1 is open --- 2901 VCC on UB+ with 210 ohm between --- UB+ whatever is connected to Batterie --- VSS on gnd --- neg input on VR2 regulated voltage --- pos input on [R9..R11.R16] voltage div net --- all leds always in indicating state"
- note added: "connected to Batterie is internal Battery, evtl. external Batterie or not impossible external Battery loader"
- note added: "no power adapter connected, S2 conducting: --- same as with power adapter connected"
- note added: "no power adapter connected, S2 not conducting: - Uvar is on high impedance, no led on"
Changed lines of the file:
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@@
 <text x="-7.62" y="83.82" size="3.81" layer="91">?</text>
 <text x="-45.72" y="27.94" size="1.778" layer="91">protection</text>
+<text x="132.08" y="104.14" size="1.778" layer="91">no power adapter connected, S2 not conducting:
+- Uvar is on high impedance, no led on</text>
+<text x="132.08" y="53.34" size="1.778" layer="91">220V power adapter connected with matching
+adapter, S2 pressed (Uvar1 exactly 0):
+--- Uvar on gnd because Q1 is open
+--- 2901 VCC on UB+ with 210 ohm between
+--- UB+ whatever is connected to Batterie
+--- VSS on gnd
+--- neg input on VR2 regulated voltage
+--- pos input on [R9..R11.R16] voltage div net
+--- all leds always in indicating state</text>
+<text x="132.08" y="93.98" size="1.778" layer="91">no power adapter connected, S2 conducting:
+---  same as with power adapter connected</text>
+<text x="-96.52" y="7.62" size="1.778" layer="91">connected to Batterie is
+internal Battery, evtl.
+external Batterie or not
+impossible external
+Battery loader</text>
 </plain>
 <instances>
@@
 <wire x1="45.72" y1="66.04" x2="45.72" y2="76.2" width="0.1524" layer="91"/>
 <label x="-12.7" y="93.98" size="1.778" layer="95"/>
-<label x="96.52" y="99.06" size="1.778" layer="95"/>
-<label x="-17.78" y="76.2" size="1.778" layer="95" rot="R90"/>
+<label x="96.52" y="93.98" size="1.778" layer="95"/>
+<label x="-15.24" y="76.2" size="1.778" layer="95" rot="R90"/>
 <label x="58.42" y="-12.7" size="1.778" layer="95"/>
 <wire x1="83.82" y1="91.44" x2="83.82" y2="93.98" width="0.1524" layer="91"/>
@@
 </schematic>
 </drawing>
+<compatibility>
+<note version="6.3" minversion="6.2.2" severity="warning">
+Since Version 6.2.2 text objects can contain more than one line,
+which will not be processed correctly with this version.
+</note>
+</compatibility>
 </eagle>

Commit message: reg save
Parts:
- removed R18: xk?, resistor:R-EU_0309/10
Connections:
- removed net N$26: R18.1, S2.S
- net N$28: no longer R18.2
Other:
- note removed: "?"
- note removed: "load simulation for battery test on leds ???"
- moved on the sheet: J2-2, S2
Changed lines of the file:
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@@
 <part name="SUPPLY7" library="supply2" deviceset="-UB" device=""/>
 <part name="SUPPLY8" library="supply2" deviceset="GND" device=""/>
-<part name="R18" library="resistor" deviceset="R-EU_" device="0309/10" value="xk?"/>
 <part name="SUPPLY2" library="supply2" deviceset="-UB" device=""/>
 <part name="SUPPLY9" library="supply2" deviceset="+15V" device=""/>
@@
 <text x="35.56" y="114.3" size="1.778" layer="91">======</text>
 <text x="50.8" y="5.08" size="1.778" layer="91" rot="R90">======</text>
-<text x="15.24" y="78.74" size="1.778" layer="91">push button</text>
-<text x="15.24" y="83.82" size="1.778" layer="91">load simulation for battery test on leds ???</text>
-<text x="-7.62" y="83.82" size="3.81" layer="91">?</text>
+<text x="12.7" y="78.74" size="1.778" layer="91">push button</text>
 <text x="-45.72" y="27.94" size="1.778" layer="91">protection</text>
 <text x="132.08" y="104.14" size="1.778" layer="91">no power adapter connected, S2 not conducting:
@@
 <instance part="R16" gate="G$1" x="-38.1" y="48.26" rot="R90"/>
 <instance part="J2" gate="-1" x="10.16" y="55.88" rot="R90"/>
-<instance part="J2" gate="-2" x="5.08" y="55.88" rot="R90"/>
+<instance part="J2" gate="-2" x="2.54" y="55.88" rot="R90"/>
 <instance part="D9" gate="1" x="-20.32" y="116.84"/>
 <instance part="IC1" gate="A1" x="7.62" y="114.3"/>
@@
 <instance part="D8" gate="1" x="-48.26" y="27.94" rot="R270"/>
 <instance part="SUPPLY5" gate="G$1" x="-71.12" y="30.48"/>
-<instance part="SUPPLY6" gate="G$1" x="104.14" y="0"/>
+<instance part="SUPPLY6" gate="G$1" x="104.14" y="-5.08"/>
 <instance part="BATTERY" gate="-1" x="-73.66" y="27.94" rot="R180"/>
 <instance part="BATTERY" gate="-2" x="-73.66" y="38.1" rot="R180"/>
 <instance part="SUPPLY7" gate="G$1" x="-71.12" y="40.64" rot="R180"/>
 <instance part="SUPPLY8" gate="GND" x="-55.88" y="35.56"/>
-<instance part="R18" gate="G$1" x="-2.54" y="83.82" rot="R90"/>
 <instance part="SUPPLY2" gate="G$1" x="-55.88" y="78.74" rot="R270"/>
 <instance part="SUPPLY9" gate="+15V" x="-33.02" y="119.38"/>
-<instance part="S2" gate="BEF1" x="7.62" y="81.28" rot="MR270"/>
+<instance part="S2" gate="BEF1" x="5.08" y="81.28" rot="MR270"/>
 <instance part="SUPPLY4" gate="G$1" x="-10.16" y="-5.08"/>
 </instances>
@@
 <junction x="53.34" y="116.84"/>
 <pinref part="SUPPLY6" gate="G$1" pin="+UB"/>
-<wire x1="124.46" y1="-2.54" x2="104.14" y2="-2.54" width="0.1524" layer="91"/>
-<wire x1="124.46" y1="-2.54" x2="124.46" y2="116.84" width="0.1524" layer="91"/>
+<wire x1="124.46" y1="-7.62" x2="104.14" y2="-7.62" width="0.1524" layer="91"/>
+<wire x1="124.46" y1="-7.62" x2="124.46" y2="116.84" width="0.1524" layer="91"/>
 <wire x1="124.46" y1="116.84" x2="53.34" y2="116.84" width="0.1524" layer="91"/>
 <label x="114.3" y="116.84" size="1.778" layer="95"/>
-<wire x1="104.14" y1="-2.54" x2="88.9" y2="-2.54" width="0.1524" layer="91"/>
+<wire x1="104.14" y1="-7.62" x2="88.9" y2="-7.62" width="0.1524" layer="91"/>
 <pinref part="R15" gate="G$1" pin="1"/>
-<wire x1="88.9" y1="-2.54" x2="86.36" y2="-2.54" width="0.1524" layer="91"/>
-<wire x1="88.9" y1="2.54" x2="88.9" y2="-2.54" width="0.1524" layer="91"/>
-<wire x1="86.36" y1="-2.54" x2="81.28" y2="-2.54" width="0.1524" layer="91" curve="-180"/>
-<wire x1="81.28" y1="-2.54" x2="66.04" y2="-2.54" width="0.1524" layer="91"/>
+<wire x1="88.9" y1="-7.62" x2="86.36" y2="-7.62" width="0.1524" layer="91"/>
+<wire x1="88.9" y1="2.54" x2="88.9" y2="-7.62" width="0.1524" layer="91"/>
+<wire x1="86.36" y1="-7.62" x2="81.28" y2="-7.62" width="0.1524" layer="91" curve="180"/>
+<wire x1="81.28" y1="-7.62" x2="66.04" y2="-7.62" width="0.1524" layer="91"/>
 <pinref part="VR2" gate="G$1" pin="S"/>
 <pinref part="VR2" gate="G$1" pin="A"/>
 <wire x1="66.04" y1="5.08" x2="66.04" y2="0" width="0.1524" layer="91"/>
 <wire x1="66.04" y1="0" x2="60.96" y2="0" width="0.1524" layer="91"/>
-<wire x1="66.04" y1="-2.54" x2="66.04" y2="0" width="0.1524" layer="91"/>
-<wire x1="66.04" y1="-7.62" x2="66.04" y2="-2.54" width="0.1524" layer="91"/>
+<wire x1="66.04" y1="-7.62" x2="66.04" y2="0" width="0.1524" layer="91"/>
 <label x="71.12" y="-5.08" size="1.778" layer="95"/>
 <wire x1="15.24" y1="-7.62" x2="35.56" y2="-7.62" width="0.1524" layer="91"/>
@@
 <label x="58.42" y="-12.7" size="1.778" layer="95"/>
 <wire x1="83.82" y1="91.44" x2="83.82" y2="93.98" width="0.1524" layer="91"/>
-<wire x1="119.38" y1="93.98" x2="119.38" y2="0" width="0.1524" layer="91"/>
+<wire x1="119.38" y1="93.98" x2="119.38" y2="-5.08" width="0.1524" layer="91"/>
 <label x="119.38" y="22.86" size="1.778" layer="95" rot="R90"/>
 <wire x1="83.82" y1="-12.7" x2="119.38" y2="-12.7" width="0.1524" layer="91"/>
-<wire x1="119.38" y1="-12.7" x2="119.38" y2="-5.08" width="0.1524" layer="91"/>
-<wire x1="119.38" y1="-5.08" x2="119.38" y2="0" width="0.1524" layer="91" curve="-180"/>
+<wire x1="119.38" y1="-12.7" x2="119.38" y2="-10.16" width="0.1524" layer="91"/>
+<wire x1="119.38" y1="-10.16" x2="119.38" y2="-5.08" width="0.1524" layer="91" curve="-180"/>
 <wire x1="48.26" y1="-12.7" x2="48.26" y2="0" width="0.1524" layer="91"/>
 <pinref part="D10" gate="1" pin="C"/>
@@
 <junction x="83.82" y="93.98"/>
 <pinref part="J2" gate="-2" pin="S"/>
-<wire x1="5.08" y1="48.26" x2="5.08" y2="53.34" width="0.1524" layer="91"/>
-<wire x1="5.08" y1="48.26" x2="-15.24" y2="48.26" width="0.1524" layer="91"/>
+<wire x1="2.54" y1="48.26" x2="2.54" y2="53.34" width="0.1524" layer="91"/>
+<wire x1="2.54" y1="48.26" x2="-15.24" y2="48.26" width="0.1524" layer="91"/>
 </segment>
 </net>
@@
 <net name="N$28" class="0">
 <segment>
-<pinref part="R18" gate="G$1" pin="2"/>
-<wire x1="-2.54" y1="88.9" x2="12.7" y2="88.9" width="0.1524" layer="91"/>
-<wire x1="10.16" y1="55.88" x2="10.16" y2="71.12" width="0.1524" layer="91"/>
-<wire x1="10.16" y1="71.12" x2="12.7" y2="71.12" width="0.1524" layer="91"/>
+<wire x1="10.16" y1="55.88" x2="10.16" y2="81.28" width="0.1524" layer="91"/>
 <pinref part="S2" gate="BEF1" pin="P"/>
-<wire x1="12.7" y1="71.12" x2="12.7" y2="81.28" width="0.1524" layer="91"/>
-<wire x1="12.7" y1="88.9" x2="12.7" y2="81.28" width="0.1524" layer="91"/>
 </segment>
 </net>
 <net name="N$5" class="0">
 <segment>
-<wire x1="5.08" y1="55.88" x2="5.08" y2="78.74" width="0.1524" layer="91"/>
-</segment>
-</net>
-<net name="N$26" class="0">
-<segment>
-<pinref part="R18" gate="G$1" pin="1"/>
-<pinref part="S2" gate="BEF1" pin="S"/>
-<wire x1="-2.54" y1="78.74" x2="2.54" y2="78.74" width="0.1524" layer="91"/>
-</segment>
-</net>
+<wire x1="2.54" y1="55.88" x2="2.54" y2="78.74" width="0.1524" layer="91"/>
+</segment>
+</net>

Commit message: reg save
Other:
- note added: "connected to Batterie is internal Battery, evtl. external Batterie or external Battery loader (LIMA)"
- note added: "leds"
- note added: "load current/voltage"
- note added: "using power adapter for load ================== where is a current limitingresistor? what is the loadcurrent? what the load volatage?"
- note removed: "connected to Batterie is internal Battery, evtl. external Batterie or not impossible external Battery loader"
Changed lines of the file:
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@@
 <text x="12.7" y="78.74" size="1.778" layer="91">push button</text>
 <text x="-45.72" y="27.94" size="1.778" layer="91">protection</text>
-<text x="132.08" y="104.14" size="1.778" layer="91">no power adapter connected, S2 not conducting:
+<text x="134.62" y="104.14" size="1.778" layer="91">no power adapter connected, S2 not conducting:
 - Uvar is on high impedance, no led on</text>
-<text x="132.08" y="53.34" size="1.778" layer="91">220V power adapter connected with matching
+<text x="134.62" y="63.5" size="1.778" layer="91">220V power adapter connected with matching
 adapter, S2 pressed (Uvar1 exactly 0):
 --- Uvar on gnd because Q1 is open
@@
 --- pos input on [R9..R11.R16] voltage div net
 --- all leds always in indicating state</text>
-<text x="132.08" y="93.98" size="1.778" layer="91">no power adapter connected, S2 conducting:
+<text x="134.62" y="93.98" size="1.778" layer="91">no power adapter connected, S2 conducting:
 ---  same as with power adapter connected</text>
-<text x="-96.52" y="7.62" size="1.778" layer="91">connected to Batterie is
+<text x="-96.52" y="5.08" size="1.778" layer="91">connected to Batterie is
 internal Battery, evtl.
-external Batterie or not
-impossible external
-Battery loader</text>
+external Batterie or
+external Battery loader
+(LIMA)</text>
+<text x="129.54" y="45.72" size="3.302" layer="91">load current/voltage</text>
+<text x="129.54" y="111.76" size="3.302" layer="91">leds</text>
+<text x="134.62" y="30.48" size="1.778" layer="91">using power adapter for load
+==================
+where is a current limitingresistor?
+what is the loadcurrent?
+what the load volatage?</text>
 </plain>
 <instances>
